File: pic32ak_fe.brd (EAGLE design)
At the start: 160 x 100 mm, 3 parts, among them U1 PIC32AK1216GC41064-E/PT

Commit message: up
Connections:
- net DIS_CS: now also U1.62; no longer U1.32
- net SCK1: now also U1.63; no longer U1.31
- net SCK2: now also U1.31
- net SDI2: now also U1.32
- net SDO1: now also U1.50; no longer U1.34
- net SDO2: now also U1.34
Routing:
- net SRAM_CS: track 68.6 -> 40.1 mm
- net VSS: track 20.6 -> 43.2 mm, vias 7 -> 6
- net VDD: track 101.4 -> 115.0 mm, vias 0 -> 3
- net SCK1: track 13.2 -> 0.00 mm
- net SCK2: track 28.6 -> 40.0 mm, vias 1 -> 0
- net DIS_CS: track 11.3 -> 0.00 mm
- net SDI1: track 29.4 -> 19.4 mm, vias 0 -> 1
- net SDO1: track 25.9 -> 34.0 mm
- net SDI2: track 23.2 -> 29.7 mm, vias 1 -> 3
- net SDO2: track 30.5 -> 26.5 mm
- net DIS_MODE: track 23.8 -> 20.5 mm, vias 0 -> 1

Commit message: up
Parts:
- removed SRAM: SRAM, con-lstb:MA10-1
- added C1, C14, C16, C2, C3, C4, C5, C6: 1000pf, rcl:C0603
- added C10, C11, C12, C13, C15, C7, C8, C9: 0.1uf, rcl:C0603
- added C17, C18, C19, C20: 10uf, rcl:C0805
- added E1: LI0603G121R-10, LI0603G121R-10:FB_LI0603G121R-10
- added IC1: NCP1117LPST33T3G, NCP1117LPST33T3G:SOT230P700X180-4N
- added R1: 100 ohm, rcl:R0805
- added R2: 10K ohm, rcl:R0805
- added U2: IS66WVS4M8BLL-104NLI, iss66:SOIC8_150MIL_N_ISI
- added Y1: KC2520Z8.00000C1KX00, KC2520Z8.00000C1KX00:KC2520Z800000C1KX00
Connections:
- new net 8MHZ_CLK: U1.38, Y1.3
- new net AVDD: C3.1, C9.2, E1.2, U1.11
- new net MCLR: R1.1, U1.64
- new net N$1: C16.1, R1.2, R2.1
- new net VIN: C17.1, IC1.3
- net SCK1: now also U2.6
- net SCK2: no longer SRAM.3
- net SDI1: now also U2.2
- net SDI2: no longer SRAM.1
- net SDO1: now also U2.5
- net SDO2: no longer SRAM.2, U1.30
- net SRAM_CS: now also U2.1; no longer SRAM.5
- net VDD: now also C1.1, C10.2, C11.2, C12.2, C13.1, C14.1, C15.2, C18.1, C19.2, C2.1, C20.1, C4.1, C5.1, C6.1, C7.2, C8.2, E1.1, IC1.2, IC1.4, R2.2, U2.8, Y1.1, Y1.4; no longer SRAM.7, U1.11
- net VSS: now also C1.2, C10.1, C11.1, C12.1, C13.2, C14.2, C15.1, C16.2, C17.2, C18.2, C19.1, C2.2, C20.2, C3.2, C4.2, C5.2, C6.2, C7.1, C8.1, C9.1, IC1.1, U2.4, Y1.2; no longer SRAM.8
Routing:
- net VDD: track 115.0 -> 208.5 mm, vias 3 -> 6
- net VSS: track 43.2 -> 108.9 mm, vias 6 -> 7
- net SCK1: track 0.00 -> 53.8 mm, vias 0 -> 2
- net DIS_CS: track 0.00 -> 37.8 mm, vias 0 -> 1
- net SRAM_CS: track 40.1 -> 12.2 mm, vias 0 -> 1
- net SDO2: track 26.5 -> 0.00 mm, vias 1 -> 0
- net MCLR: track 0.00 -> 25.1 mm, vias 0 -> 1
- net SCK2: track 40.0 -> 15.0 mm, vias 0 -> 2
- net SDI2: track 29.7 -> 8.43 mm, vias 3 -> 0
- net AVDD: track 0.00 -> 11.7 mm, vias 0 -> 1
- net 8MHZ_CLK: track 0.00 -> 11.4 mm, vias 0 -> 1
- net SDI1: track 19.4 -> 30.5 mm
- net SDO1: track 34.0 -> 42.5 mm, vias 0 -> 2
- net N$1: track 0.00 -> 5.90 mm
- net VIN: track 0.00 -> 5.24 mm, vias 0 -> 1
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- added copper zone on layer 1, net VDD

Commit message: up
Parts:
- added ICSP: ICSP, pinhead:1X06/90
- added LED2, LED3, LED4: (no value), led:CHIP-LED0603
- added POWER: POWER, led:CHIP-LED0603
- added R3, R4, R5, R6: 1K ohm, rcl:R0805
Connections:
- new net DLED: R5.2, U1.53
- new net HLED: R6.2, U1.49
- new net N$2: POWER.A, R3.1
- new net N$3: LED2.A, R4.1
- new net N$4: LED3.A, R5.1
- new net N$5: LED4.A, R6.1
- new net N$8: U1.52
- new net PGC: ICSP.5, U1.3
- new net PGD: ICSP.4, U1.1
- new net RLED: R4.2, U1.51
- net MCLR: now also ICSP.1
- net VDD: now also ICSP.2, R3.2
- net VSS: now also ICSP.3, LED2.C, LED3.C, LED4.C, POWER.C
Routing:
- net PGD: track 0.00 -> 67.8 mm, vias 0 -> 1
- net PGC: track 0.00 -> 67.5 mm, vias 0 -> 3
- net VSS: track 108.9 -> 61.8 mm, vias 7 -> 18
- net MCLR: track 25.1 -> 59.9 mm, vias 1 -> 4
- net DLED: track 0.00 -> 31.2 mm, vias 0 -> 2
- net HLED: track 0.00 -> 31.0 mm, vias 0 -> 2
- net RLED: track 0.00 -> 28.0 mm, vias 0 -> 2
- net VDD: track 208.5 -> 192.5 mm, vias 6 -> 18
- net SDO1: track 42.5 -> 49.1 mm
- net DIS_CS: track 37.8 -> 32.3 mm, vias 1 -> 4
- net N$3: track 0.00 -> 4.93 mm
- net SCK1: track 53.8 -> 49.8 mm, vias 2 -> 3
- net SDI1: track 30.5 -> 33.3 mm, vias 1 -> 3
- net N$5: track 0.00 -> 2.11 mm
- net N$4: track 0.00 -> 2.11 mm
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
Commit message: up
Parts:
- added FUSE: 0 ohm, rcl:R0805
- added J1, J2, J3, J4: CONBNC001, CONBNC001:CONBNC001
- added MISC_ANA: MISC_ANA, pinhead:1X06/90
- added R10, R7, R8, R9: 50 ohm, rcl:R0805
- added S1: PTS635SL50LFS, PTS635SL50LFS:PTS635SL50LFS
- added TP1, TP2, TP3, TP4, TP5, TP6: PTR1PAD1-13, testpad:P1-13
- added TP10, TP11, TP12, TP7, TP8, TP9: PTR1PAD1-20, testpad:P1-20
- added X1: 22-23-2021, con-molex:22-23-2021
- LED2: value (none) -> rled
- LED3: value (none) -> dled
- LED4: value (none) -> hled
Connections:
- removed net N$1: C16.1, R1.2, R2.1
- removed net N$8: U1.52
- removed net PGC: ICSP.5, U1.3
- new net AD1AN6: J1.1, R7.2, U1.2
- new net AD2AN7: J2.1, R8.2, U1.9
- new net OA2IN: J3.1, R9.2, U1.22
- new net OA2OUT: J4.1, R10.2, U1.20
- new net PGC_DAC: ICSP.5, MISC_ANA.2, U1.3
- new net RESET_SW: C16.1, R1.2, R2.1, S1.2, TP12.TP
- new net VIN_PWR: FUSE.2, X1.2
- net 8MHZ_CLK: now also TP6.TP
- net AVDD: now also MISC_ANA.6
- net DLED: now also TP8.TP
- net HLED: now also TP9.TP
- net RLED: now also TP7.TP
- net SCK1: no longer U2.6
- net SCK2: now also TP2.TP, U2.6; no longer U1.45
- net SDI1: no longer U2.2
- net SDI2: now also TP4.TP, U2.3
- net SDO1: no longer U2.5
- net SDO2: now also TP1.TP, U2.5
- net SRAM_CS: now also TP5.TP
- net VDD: now also TP10.TP
- net VIN: now also FUSE.1
- net VSS: now also J1.2, J1.3, J1.4, J1.5, J2.2, J2.3, J2.4, J2.5, J3.2, J3.3, J3.4, J3.5, J4.2, J4.3, J4.4, J4.5, MISC_ANA.1, R10.1, R7.1, R8.1, R9.1, S1.1, TP11.TP, TP3.TP, X1.1
Routing:
- net VDD: track 192.5 -> 25.8 mm, vias 18 -> 0
- net PGD: track 67.8 -> 0.00 mm, vias 1 -> 0
- net PGC: track 67.5 -> 0.00 mm, vias 3 -> 0
- net MCLR: track 59.9 -> 0.00 mm, vias 4 -> 0
- net SCK1: track 49.8 -> 0.00 mm, vias 3 -> 0
- net SDO1: track 49.1 -> 0.00 mm, vias 2 -> 0
- net SDI1: track 33.3 -> 0.00 mm, vias 3 -> 0
- net DIS_CS: track 32.3 -> 0.00 mm, vias 4 -> 0
- net DLED: track 31.2 -> 0.00 mm, vias 2 -> 0
- net HLED: track 31.0 -> 0.00 mm, vias 2 -> 0
- net RLED: track 28.0 -> 0.00 mm, vias 2 -> 0
- net DIS_MODE: track 21.3 -> 0.00 mm, vias 1 -> 0
- net DIS_RESET: track 17.9 -> 0.00 mm, vias 1 -> 0
- net VSS: track 61.8 -> 44.9 mm, vias 18 -> 5
- net SCK2: track 13.1 -> 0.00 mm, vias 2 -> 0
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
Commit message: up
Parts:
- added J5: 22-27-2021-02, con-molex:6410-02
- added TP13, TP14, TP15, TP16, TP17, TP18: PTR1PAD1-13, testpad:P1-13
- moved MISC_ANA 17.7 mm to (53.3, 47.0)
Connections:
- net RESET_SW: now also J5.2
- net SDI2: no longer U1.36
- net VDD: now also TP13.TP, TP14.TP, TP15.TP
- net VSS: now also J5.1, TP16.TP, TP17.TP, TP18.TP
Routing:
- net AD1AN6: track 0.00 -> 2.18 mm
- net SDI2: track 1.82 -> 0.00 mm

Commit message: up
Parts:
- removed TP7, TP8: PTR1PAD1-20, testpad:P1-20
- moved TP10 29.9 mm to (72.4, 33.0)
- moved TP6 12.6 mm to (34.3, 19.1)
- moved TP9 5.08 mm to (53.3, 26.7)
Connections:
- net DLED: no longer TP8.TP
- net RLED: no longer TP7.TP
Routing:
- net VDD: track 25.8 -> 214.1 mm, vias 0 -> 15
- net PGC_DAC: track 0.00 -> 94.6 mm, vias 0 -> 2
- net PGD: track 0.00 -> 69.1 mm, vias 0 -> 5
- net OA2IN: track 0.00 -> 62.6 mm, vias 0 -> 2
- net AVDD: track 6.20 -> 67.9 mm, vias 0 -> 4
- net MCLR: track 0.00 -> 59.1 mm, vias 0 -> 7
- net RESET_SW: track 0.00 -> 53.2 mm, vias 0 -> 2
- net AD1AN6: track 2.18 -> 47.0 mm
- net OA2OUT: track 0.00 -> 43.1 mm, vias 0 -> 2
- net SDO1: track 0.00 -> 34.5 mm, vias 0 -> 2
- net HLED: track 0.00 -> 33.8 mm, vias 0 -> 3
- net RLED: track 0.00 -> 32.7 mm, vias 0 -> 2
- net AD2AN7: track 0.00 -> 32.4 mm, vias 0 -> 2
- net DIS_CS: track 0.00 -> 32.3 mm, vias 0 -> 2
- net SCK1: track 0.00 -> 32.3 mm, vias 0 -> 2
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
Commit message: up
Parts:
- renumbered J5 to R_RESET, TP9 to TEST_P0, X1 to VIN_5+

Commit message: up
Parts:
- added J5: 5227222-3, 5227222-3:52272223
Connections:
- net PGC_DAC: now also J5.1
- net VSS: now also J5.2
Routing:
- net PGC_DAC: track 94.6 -> 123.7 mm
Changed lines of the file:
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@@
 <grid distance="50" unitdist="mil" unit="mil" style="lines" multiple="1" display="no" altdistance="5" altunitdist="mil" altunit="mil"/>
 <layers>
-<layer number="1" name="Top" color="4" fill="1" visible="no" active="yes"/>
-<layer number="2" name="Route2" color="16" fill="1" visible="no" active="yes"/>
-<layer number="3" name="Route3" color="17" fill="1" visible="no" active="yes"/>
+<layer number="1" name="Top" color="4" fill="1" visible="yes" active="yes"/>
+<layer number="2" name="Route2" color="16" fill="1" visible="yes" active="yes"/>
+<layer number="3" name="Route3" color="17" fill="1" visible="yes" active="yes"/>
 <layer number="4" name="Route4" color="18" fill="1" visible="no" active="no"/>
 <layer number="5" name="Route5" color="19" fill="1" visible="no" active="no"/>
@@
 <layer number="13" name="Route13" color="21" fill="1" visible="no" active="no"/>
 <layer number="14" name="Route14" color="22" fill="1" visible="no" active="no"/>
-<layer number="15" name="Route15" color="23" fill="1" visible="no" active="yes"/>
+<layer number="15" name="Route15" color="23" fill="1" visible="yes" active="yes"/>
 <layer number="16" name="Bottom" color="1" fill="1" visible="yes" active="yes"/>
 <layer number="17" name="Pads" color="2" fill="1" visible="yes" active="yes"/>
@@
 <layer number="19" name="Unrouted" color="6" fill="1" visible="yes" active="yes"/>
 <layer number="20" name="Dimension" color="24" fill="1" visible="yes" active="yes"/>
-<layer number="21" name="tPlace" color="7" fill="1" visible="no" active="yes"/>
+<layer number="21" name="tPlace" color="7" fill="1" visible="yes" active="yes"/>
 <layer number="22" name="bPlace" color="7" fill="1" visible="yes" active="yes"/>
-<layer number="23" name="tOrigins" color="15" fill="1" visible="no" active="yes"/>
+<layer number="23" name="tOrigins" color="15" fill="1" visible="yes" active="yes"/>
 <layer number="24" name="bOrigins" color="15" fill="1" visible="yes" active="yes"/>
-<layer number="25" name="tNames" color="7" fill="1" visible="no" active="yes"/>
+<layer number="25" name="tNames" color="7" fill="1" visible="yes" active="yes"/>
 <layer number="26" name="bNames" color="7" fill="1" visible="yes" active="yes"/>
 <layer number="27" name="tValues" color="7" fill="1" visible="no" active="yes"/>
@@
 <layer number="37" name="tTest" color="7" fill="1" visible="no" active="yes"/>
 <layer number="38" name="bTest" color="7" fill="1" visible="no" active="yes"/>
-<layer number="39" name="tKeepout" color="4" fill="11" visible="no" active="yes"/>
+<layer number="39" name="tKeepout" color="4" fill="11" visible="yes" active="yes"/>
 <layer number="40" name="bKeepout" color="1" fill="11" visible="yes" active="yes"/>
-<layer number="41" name="tRestrict" color="4" fill="10" visible="no" active="yes"/>
+<layer number="41" name="tRestrict" color="4" fill="10" visible="yes" active="yes"/>
 <layer number="42" name="bRestrict" color="1" fill="10" visible="yes" active="yes"/>
 <layer number="43" name="vRestrict" color="2" fill="10" visible="no" active="yes"/>
@@
 <layer number="48" name="Document" color="7" fill="1" visible="no" active="yes"/>
 <layer number="49" name="Reference" color="7" fill="1" visible="no" active="yes"/>
-<layer number="51" name="tDocu" color="7" fill="1" visible="no" active="yes"/>
+<layer number="51" name="tDocu" color="7" fill="1" visible="yes" active="yes"/>
 <layer number="52" name="bDocu" color="7" fill="1" visible="yes" active="yes"/>
 <layer number="88" name="SimResults" color="9" fill="1" visible="no" active="no"/>
@@
 <attribute name="VALUE" x="44.45" y="67.31" size="0.0254" layer="27"/>
 </element>
+<element name="J5" library="5227222-3" package="52272223" value="5227222-3" x="71.12" y="60.96" smashed="yes">
+<attribute name="DESCRIPTION" value="Body Features: Body Material Finish Passivated | Body Plating Material Nickel | Body Material Polyester, PBT | Configuration Features: Number of Coaxial Contacts 1 | PCB Mount Orientation Vertical | Number of Positions 1 | Contact Features: RF Connector Center Contact Material Phosphor Bronze | RF Connector Center Contact Plating Thickness 889 MICIN | RF Connector Center Contact Underplating Material Nickel | RF Connector Center Contact Plating Material Gold | Dimensions: Profile Height from PCB 1.375 INCH " x="71.12" y="60.96" size="1.778" layer="27" display="off"/>
+<attribute name="HEIGHT" value="35.57mm" x="71.12" y="60.96" size="1.778" layer="27" display="off"/>
+<attribute name="MANUFACTURER_NAME" value="TE Connectivity" x="71.12" y="60.96" size="1.778" layer="27" display="off"/>
+<attribute name="MANUFACTURER_PART_NUMBER" value="5227222-3" x="71.12" y="60.96" size="1.778" layer="27" display="off"/>
+<attribute name="MOUSER_PART_NUMBER" value="571-5227222-3" x="71.12" y="60.96" size="1.778" layer="27" display="off"/>
+<attribute name="MOUSER_PRICE-STOCK" value="https://www.mouser.co.uk/ProductDetail/TE-Connectivity/5227222-3?qs=GSeC4G%252BEqEW87SYw9J0%252BtA%3D%3D" x="71.12" y="60.96" size="1.778" layer="27" display="off"/>
+<attribute name="NAME" x="71.12" y="57.045" size="1.27" layer="25" align="center"/>
+<attribute name="VALUE" x="71.12" y="60.855" size="1.27" layer="27" align="center"/>
+</element>
 </elements>
 <signals>
@@
 <via x="16.8275" y="14.605" extent="1-16" drill="0.35"/>
 <via x="27.305" y="24.765" extent="1-16" drill="0.35"/>
+<contactref element="J5" pad="2"/>
 </signal>
 <signal name="SDI1">
@@
 <via x="12.3825" y="27.6225" extent="1-16" drill="0.35"/>
 <via x="63.8175" y="9.8425" extent="1-16" drill="0.35"/>
+<contactref element="J5" pad="1"/>
+<wire x1="70.0278" y1="60.96" x2="71.12" y2="60.96" width="0.1524" layer="1"/>
+<wire x1="67.1322" y1="58.0644" x2="70.0278" y2="60.96" width="0.1524" layer="1"/>
+<wire x1="64.77" y1="58.0644" x2="67.1322" y2="58.0644" width="0.1524" layer="1"/>
+<wire x1="49.7586" y1="43.053" x2="64.77" y2="58.0644" width="0.1524" layer="1"/>
+<wire x1="49.7586" y1="43.053" x2="49.53" y2="43.18" width="0.1524" layer="1"/>
 </signal>
 <signal name="N$2">
