File: pic32ak_fe.brd (EAGLE design)
At the start: 119.4 x 77.1 mm, 87 parts, among them IC1 NCP1117LPST33T3G, IC2 SFH6916, J1 CONBNC001, J2 CONBNC001, J3 CONBNC001, J4 CONBNC001, J5 5227222-3, SW1 PTS635SL50LFS, SW2 PTS635SL50LFS, U1 PIC32AK1216GC41064-E/PT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

Commit message: up
Connections:
- removed net RD8: MISC_ANA.3, U1.58
- new net RB1: MISC_ANA.3, U1.21
- net SCK3: now also U1.58; no longer U1.21
- net SDI2: no longer U2.3
Routing:
- net RB1: track 0.00 -> 70.8 mm, vias 0 -> 3
- net RD8: track 40.1 -> 0.00 mm
- net SCK3: track 84.8 -> 84.3 mm, vias 4 -> 3
Changed lines of the file:
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@@
 <layer number="41" name="tRestrict" color="4" fill="10" visible="yes" active="yes"/>
 <layer number="42" name="bRestrict" color="1" fill="10" visible="yes" active="yes"/>
-<layer number="43" name="vRestrict" color="2" fill="10" visible="yes" active="yes"/>
+<layer number="43" name="vRestrict" color="2" fill="10" visible="no" active="yes"/>
 <layer number="44" name="Drills" color="7" fill="1" visible="no" active="yes"/>
-<layer number="45" name="Holes" color="7" fill="1" visible="yes" active="yes"/>
+<layer number="45" name="Holes" color="7" fill="1" visible="no" active="yes"/>
 <layer number="46" name="Milling" color="3" fill="1" visible="no" active="yes"/>
 <layer number="47" name="Measures" color="7" fill="1" visible="no" active="yes"/>
@@
 <signal name="SDI2">
 <contactref element="U1" pad="32"/>
-<contactref element="U2" pad="3"/>
-<contactref element="TP4" pad="TP"/>
 <wire x1="25.2984" y1="15.8496" x2="24.0792" y2="15.8496" width="0.1524" layer="1"/>
 <wire x1="32.2326" y1="15.8496" x2="25.2984" y2="15.8496" width="0.1524" layer="15"/>
-<wire x1="39.1668" y1="8.9154" x2="33.7947" y2="14.2875" width="0.1524" layer="15"/>
-<wire x1="33.7947" y1="14.2875" x2="32.2326" y2="15.8496" width="0.1524" layer="15"/>
+<wire x1="39.1668" y1="8.9154" x2="33.0327" y2="15.0495" width="0.1524" layer="15"/>
+<wire x1="33.0327" y1="15.0495" x2="32.2326" y2="15.8496" width="0.1524" layer="15"/>
 <wire x1="46.9392" y1="8.9154" x2="39.1668" y2="8.9154" width="0.1524" layer="15"/>
 <wire x1="24.0792" y1="15.8496" x2="24.07" y2="15.9131" width="0.1524" layer="1"/>
+<via x="25.2984" y="15.8496" extent="1-16" drill="0.35"/>
+<contactref element="U2" pad="2"/>
+<contactref element="TP4" pad="TP"/>
+<wire x1="33.6804" y1="16.1544" x2="33.6804" y2="16.6116" width="0.1524" layer="16"/>
+<wire x1="33.6804" y1="16.6116" x2="33.655" y2="16.69415" width="0.1524" layer="16"/>
 <wire x1="46.9392" y1="8.9154" x2="46.99" y2="8.89" width="0.1524" layer="15"/>
-<wire x1="34.8996" y1="15.3924" x2="34.8996" y2="16.6878" width="0.1524" layer="16"/>
-<wire x1="33.7947" y1="14.2875" x2="34.8996" y2="15.3924" width="0.1524" layer="15"/>
-<wire x1="34.8996" y1="16.6878" x2="34.925" y2="16.69415" width="0.1524" layer="16"/>
-<via x="25.2984" y="15.8496" extent="1-16" drill="0.35"/>
-<via x="34.8996" y="15.3924" extent="1-16" drill="0.35"/>
-<contactref element="U2" pad="2"/>
-<wire x1="34.925" y1="16.69415" x2="33.655" y2="16.69415" width="0" layer="19" extent="16-16"/>
+<wire x1="33.6804" y1="15.6972" x2="33.6804" y2="16.1544" width="0.1524" layer="16"/>
+<wire x1="33.3756" y1="15.3924" x2="33.6804" y2="15.6972" width="0.1524" layer="16"/>
+<wire x1="33.0327" y1="15.0495" x2="33.3756" y2="15.3924" width="0.1524" layer="15"/>
+<wire x1="33.6804" y1="16.1544" x2="33.655" y2="16.69415" width="0.1524" layer="16"/>
+<via x="33.3756" y="15.3924" extent="1-16" drill="0.35"/>
 </signal>
 <signal name="SDO2">
@@
 <via x="22.86" y="10.3632" extent="1-16" drill="0.35"/>
 </signal>
-<signal name="SCK3">
+<signal name="RB1">
 <contactref element="U1" pad="21"/>
-<contactref element="AC1" pad="8"/>
-<wire x1="84.5058" y1="34.2138" x2="85.2678" y2="33.4518" width="0.1524" layer="1" locked="yes"/>
-<wire x1="84.5058" y1="26.0604" x2="84.5058" y2="34.2138" width="0.1524" layer="15" locked="yes"/>
-<via x="84.5058" y="34.2138" extent="1-16" drill="0.35" locked="yes"/>
-<wire x1="85.2678" y1="33.4518" x2="85.2678" y2="33.147" width="0.1524" layer="1"/>
-<wire x1="85.2678" y1="33.147" x2="85.32" y2="33.145" width="0.1524" layer="1"/>
-<wire x1="72.9996" y1="26.0604" x2="84.5058" y2="26.0604" width="0.1524" layer="15"/>
-<wire x1="68.6562" y1="21.717" x2="72.9996" y2="26.0604" width="0.1524" layer="15"/>
-<wire x1="56.2356" y1="21.717" x2="68.6562" y2="21.717" width="0.1524" layer="15"/>
 <wire x1="47.8536" y1="21.717" x2="56.2356" y2="21.717" width="0.1524" layer="1"/>
 <wire x1="46.6725" y1="22.8981" x2="47.8536" y2="21.717" width="0.1524" layer="1"/>
@@
 <wire x1="46.6344" y1="22.86" x2="46.6725" y2="22.8981" width="0.1524" layer="1"/>
 <via x="28.1178" y="22.7076" extent="1-16" drill="0.35"/>
+<contactref element="MISC_ANA" pad="3"/>
+<wire x1="52.1208" y1="42.9006" x2="52.1208" y2="43.1292" width="0.1524" layer="2"/>
+<wire x1="53.5686" y1="41.4528" x2="52.1208" y2="42.9006" width="0.1524" layer="2"/>
+<wire x1="53.5686" y1="29.8704" x2="53.5686" y2="41.4528" width="0.1524" layer="2"/>
+<wire x1="51.2826" y1="27.5844" x2="53.5686" y2="29.8704" width="0.1524" layer="2"/>
+<wire x1="51.2826" y1="25.7556" x2="51.2826" y2="27.5844" width="0.1524" layer="2"/>
+<wire x1="54.864" y1="22.1742" x2="51.2826" y2="25.7556" width="0.1524" layer="2"/>
+<wire x1="55.3974" y1="22.1742" x2="54.864" y2="22.1742" width="0.1524" layer="2"/>
+<wire x1="55.9308" y1="21.6408" x2="55.3974" y2="22.1742" width="0.1524" layer="2"/>
+<wire x1="56.1594" y1="21.6408" x2="55.9308" y2="21.6408" width="0.1524" layer="2"/>
+<wire x1="56.2356" y1="21.717" x2="56.1594" y2="21.6408" width="0.1524" layer="2"/>
+<wire x1="52.1208" y1="43.1292" x2="52.07" y2="43.18" width="0.1524" layer="2"/>
 </signal>
 <signal name="SDI3">
@@
 <via x="48.4632" y="39.7002" extent="1-16" drill="0.35"/>
 </signal>
-<signal name="RD8">
+<signal name="SCK3">
 <contactref element="U1" pad="58"/>
-<contactref element="MISC_ANA" pad="3"/>
 <wire x1="19.5834" y1="29.0322" x2="19.5834" y2="27.2796" width="0.1524" layer="1"/>
 <wire x1="26.3652" y1="35.814" x2="19.5834" y2="29.0322" width="0.1524" layer="1"/>
-<wire x1="42.672" y1="35.814" x2="26.3652" y2="35.814" width="0.1524" layer="1"/>
-<wire x1="48.2346" y1="41.3766" x2="42.672" y2="35.814" width="0.1524" layer="1"/>
-<wire x1="50.292" y1="41.3766" x2="48.2346" y2="41.3766" width="0.1524" layer="1"/>
-<wire x1="52.0446" y1="43.1292" x2="50.292" y2="41.3766" width="0.1524" layer="1"/>
+<wire x1="42.5196" y1="35.814" x2="26.3652" y2="35.814" width="0.1524" layer="1"/>
 <wire x1="19.5834" y1="27.2796" x2="19.57" y2="27.2669" width="0.1524" layer="1"/>
-<wire x1="52.0446" y1="43.1292" x2="52.07" y2="43.18" width="0.1524" layer="1"/>
+<contactref element="AC1" pad="8"/>
+<wire x1="85.2678" y1="33.3756" x2="85.2678" y2="33.147" width="0.1524" layer="1"/>
+<wire x1="84.4296" y1="34.2138" x2="85.2678" y2="33.3756" width="0.1524" layer="1" locked="yes"/>
+<wire x1="81.153" y1="34.2138" x2="84.4296" y2="34.2138" width="0.1524" layer="15"/>
+<wire x1="68.0466" y1="21.1074" x2="81.153" y2="34.2138" width="0.1524" layer="15"/>
+<wire x1="55.0164" y1="21.1074" x2="68.0466" y2="21.1074" width="0.1524" layer="15"/>
+<wire x1="51.7398" y1="24.384" x2="55.0164" y2="21.1074" width="0.1524" layer="2"/>
+<wire x1="51.7398" y1="24.8412" x2="51.7398" y2="24.384" width="0.1524" layer="2"/>
+<wire x1="50.9778" y1="25.6032" x2="51.7398" y2="24.8412" width="0.1524" layer="2"/>
+<wire x1="50.9778" y1="26.2128" x2="50.9778" y2="25.6032" width="0.1524" layer="2"/>
+<wire x1="42.5196" y1="34.671" x2="50.9778" y2="26.2128" width="0.1524" layer="2"/>
+<wire x1="42.5196" y1="36.1188" x2="42.5196" y2="34.671" width="0.1524" layer="2"/>
+<wire x1="42.5196" y1="35.814" x2="42.5196" y2="36.1188" width="0.1524" layer="1"/>
+<wire x1="85.2678" y1="33.147" x2="85.32" y2="33.145" width="0.1524" layer="1"/>
+<via x="84.4296" y="34.2138" extent="1-16" drill="0.35" locked="yes"/>
+<via x="55.0164" y="21.1074" extent="1-16" drill="0.35"/>
+<via x="42.5196" y="36.1188" extent="1-16" drill="0.35"/>
 </signal>
 </signals>

Commit message: up
Parts:
- added R11, R12, R13: 100 ohm, rcl:R0805
- added TP14, TP19, TP20, TP21, TP22, TP23, TP24, TP9: PTR1PAD1-13, testpad:P1-13
Connections:
- net IMU_CS: now also TP21.TP
- net SCK2: now also R13.1
- net SCK3: now also TP14.TP
- net SDI2: now also R11.1
- net SDI3: now also TP20.TP
- net SDO2: now also R12.1
- net SDO3: now also TP9.TP
- net VSS: now also R11.2, R12.2, R13.2, TP19.TP, TP22.TP, TP23.TP, TP24.TP
Routing:
- net SCK3: track 84.3 -> 96.5 mm
- net SDO3: track 98.3 -> 108.8 mm
- net IMU_CS: track 97.7 -> 107.5 mm
- net SDI3: track 91.9 -> 98.3 mm
- net SDO2: track 27.5 -> 32.2 mm
- net SDI2: track 28.3 -> 32.5 mm
- net SCK2: track 35.5 -> 39.7 mm

Commit message: up
Parts:
- added AVDD_JUMPER: AVDD JUMPER, jumper:SJ_2
- added C27, C28: 0.1uf, rcl:C0603
- added IC3: NCP51460SN33T1G, NCP51460SN33T1G:SOT96P237X111-3N
Connections:
- new net 3.3REG: AVDD_JUMPER.1, IC3.2
- new net AVDD_IN: AVDD_JUMPER.2, C28.1, E1.1
- net VDD: now also AVDD_JUMPER.3; no longer E1.1
- net VIN: now also C27.1, IC3.1
- net VSS: now also C27.2, C28.2, IC3.3
Routing:
- net VIN: track 61.5 -> 186.1 mm, vias 2 -> 3
- net AVDD_IN: track 0.00 -> 30.2 mm, vias 0 -> 3
- net VDD: track 318.1 -> 331.5 mm
- net VSS: track 173.8 -> 182.4 mm
- net 3.3REG: track 0.00 -> 6.31 mm
Changed lines of the file:
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@@
 <attribute name="VALUE" x="42.545" y="10.16" size="1.27" layer="28" rot="MR0"/>
+</element>
+<element name="IC3" library="NCP51460SN33T1G" package="SOT96P237X111-3N" value="NCP51460SN33T1G" x="5.08" y="27.94" smashed="yes">
+<attribute name="DESCRIPTION" value="Operating Input Voltage VIN 4.2 V to 28 V; Output Current Capability of 0 to 20 mA; Output Voltage Temperature Coefficient of 18 ppm/C; Output Voltage Accuracy 1 %, for 0 C TA 100 C ; High PSRR of 68 dB at 1 kHz; Stable Without Output Capacitor; Low Quiescent Current of 140 A; Low Output Noise of 18 VRMS; Output Voltage Option: 3.3V" x="5.08" y="27.94" size="1.778" layer="27" display="off"/>
+<attribute name="HEIGHT" value="1.11mm" x="5.08" y="27.94" size="1.778" layer="27" display="off"/>
+<attribute name="MANUFACTURER_NAME" value="onsemi" x="5.08" y="27.94" size="1.778" layer="27" display="off"/>
+<attribute name="MANUFACTURER_PART_NUMBER" value="NCP51460SN33T1G" x="5.08" y="27.94" size="1.778" layer="27" display="off"/>
+<attribute name="MOUSER_PART_NUMBER" value="863-NCP51460SN33T1G" x="5.08" y="27.94" size="1.778" layer="27" display="off"/>
+<attribute name="MOUSER_PRICE-STOCK" value="https://www.mouser.co.uk/ProductDetail/onsemi/NCP51460SN33T1G?qs=yYCK2ysgWqmLP%2FSKTB%252Bdng%3D%3D" x="5.08" y="27.94" size="1.778" layer="27" display="off"/>
+<attribute name="NAME" x="5.08" y="33.02" size="1.27" layer="25" align="center"/>
+<attribute name="VALUE" x="5.08" y="27.94" size="1.27" layer="27" align="center"/>
+</element>
+<element name="AVDD_JUMPER" library="jumper" library_urn="urn:adsk.eagle:library:252" package="SJ_2" package3d_urn="urn:adsk.eagle:package:15474/1" value="AVDD JUMPER" x="5.08" y="34.29" smashed="yes" rot="R90">
+<attribute name="NAME" x="3.81" y="31.877" size="1.27" layer="25" ratio="10" rot="R90"/>
+<attribute name="POPULARITY" value="7" x="5.08" y="34.29" size="1.778" layer="27" rot="R90" display="off"/>
+<attribute name="VALUE" x="5.08" y="34.1899" size="0.02" layer="27" rot="R90"/>
+</element>
+<element name="C27" library="rcl" library_urn="urn:adsk.eagle:library:334" package="C0603" package3d_urn="urn:adsk.eagle:package:23616/2" value="0.1uf" x="5.08" y="34.29" smashed="yes" rot="MR180">
+<attribute name="NAME" x="6.985" y="34.925" size="1.27" layer="26" rot="MR180"/>
+<attribute name="POPULARITY" value="37" x="5.08" y="34.29" size="1.778" layer="28" rot="MR180" display="off"/>
+<attribute name="SPICEPREFIX" value="C" x="5.08" y="34.29" size="1.778" layer="28" rot="MR180" display="off"/>
+<attribute name="VALUE" x="4.445" y="36.195" size="1.27" layer="28" rot="MR180"/>
+</element>
+<element name="C28" library="rcl" library_urn="urn:adsk.eagle:library:334" package="C0603" package3d_urn="urn:adsk.eagle:package:23616/2" value="0.1uf" x="3.81" y="13.97" smashed="yes" rot="MR180">
+<attribute name="NAME" x="1.905" y="12.065" size="1.27" layer="26" rot="MR180"/>
+<attribute name="POPULARITY" value="37" x="3.81" y="13.97" size="1.778" layer="28" rot="MR180" display="off"/>
+<attribute name="SPICEPREFIX" value="C" x="3.81" y="13.97" size="1.778" layer="28" rot="MR180" display="off"/>
+<attribute name="VALUE" x="3.175" y="15.875" size="1.27" layer="28" rot="MR180"/>
 </element>
 </elements>
@@
 <contactref element="C5" pad="1"/>
 <contactref element="C6" pad="1"/>
-<contactref element="E1" pad="1"/>
 <wire x1="21.07" y1="15.9131" x2="21.07" y2="12.85875" width="0.2032" layer="1" locked="yes"/>
 <wire x1="21.07" y1="12.85875" x2="21.07" y2="12.22375" width="0.2032" layer="1" locked="yes"/>
@@
 <wire x1="14.6304" y1="23.3934" x2="14.6431" y2="23.34" width="0.2032" layer="1"/>
 <wire x1="14.6304" y1="23.3934" x2="14.605" y2="23.3934" width="0.2032" layer="1"/>
-<wire x1="4.3434" y1="20.4978" x2="4.3434" y2="20.3454" width="0.2032" layer="1"/>
-<wire x1="5.4102" y1="21.5646" x2="4.3434" y2="20.4978" width="0.2032" layer="1"/>
 <wire x1="6.5532" y1="22.7076" x2="5.4102" y2="21.5646" width="0.2032" layer="2"/>
 <wire x1="7.0866" y1="22.7076" x2="6.5532" y2="22.7076" width="0.2032" layer="1"/>
 <wire x1="7.62" y1="23.241" x2="7.0866" y2="22.7076" width="0.2032" layer="1"/>
-<wire x1="4.3434" y1="20.3454" x2="4.28" y2="20.32" width="0.2032" layer="1"/>
 <wire x1="7.62" y1="23.241" x2="7.62" y2="23.28" width="0.2032" layer="1"/>
 <wire x1="6.0198" y1="23.241" x2="5.1054" y2="23.241" width="0.2032" layer="16"/>
@@
 <wire x1="18.5928" y1="31.1658" x2="18.5928" y2="31.3182" width="0.2032" layer="1"/>
 <wire x1="33.2232" y1="21.4122" x2="33.17875" y2="21.34" width="0.2032" layer="1"/>
+<contactref element="AVDD_JUMPER" pad="3"/>
+<wire x1="5.334" y1="35.814" x2="5.08" y2="35.814" width="0.2032" layer="1"/>
+<wire x1="6.1722" y1="34.9758" x2="5.334" y2="35.814" width="0.2032" layer="1"/>
+<wire x1="6.1722" y1="29.0322" x2="6.1722" y2="34.9758" width="0.2032" layer="1"/>
+<wire x1="5.4102" y1="28.2702" x2="6.1722" y2="29.0322" width="0.2032" layer="1"/>
+<wire x1="5.4102" y1="21.5646" x2="5.4102" y2="28.2702" width="0.2032" layer="1"/>
 </signal>
 <signal name="VSS" class="1">
@@
 <wire x1="4.2672" y1="17.7546" x2="4.23" y2="17.78" width="0.2032" layer="1"/>
 <wire x1="7.62" y1="12.7254" x2="7.62" y2="12.7" width="0.2032" layer="1"/>
-<wire x1="9.2964" y1="24.9174" x2="7.62" y2="24.9174" width="0.2032" layer="1"/>
+<wire x1="9.2964" y1="24.9174" x2="8.3058" y2="24.9174" width="0.2032" layer="1"/>
+<wire x1="8.3058" y1="24.9174" x2="7.62" y2="24.9174" width="0.2032" layer="1"/>
 <wire x1="10.3632" y1="23.8506" x2="9.2964" y2="24.9174" width="0.2032" layer="1"/>
 <wire x1="7.62" y1="24.9174" x2="7.62" y2="24.98" width="0.2032" layer="1"/>
@@
 <contactref element="R11" pad="2"/>
 <contactref element="R12" pad="2"/>
+<contactref element="IC3" pad="3"/>
+<wire x1="7.0104" y1="27.8892" x2="6.3246" y2="27.8892" width="0.2032" layer="1"/>
+<wire x1="8.3058" y1="26.5938" x2="7.2898" y2="27.6098" width="0.2032" layer="1"/>
+<wire x1="7.2898" y1="27.6098" x2="7.0104" y2="27.8892" width="0.2032" layer="1"/>
+<wire x1="8.3058" y1="24.9174" x2="8.3058" y2="26.5938" width="0.2032" layer="1"/>
+<wire x1="6.3246" y1="27.8892" x2="6.28" y2="27.94" width="0.2032" layer="1"/>
+<contactref element="C27" pad="2"/>
+<contactref element="C28" pad="2"/>
+<wire x1="7.62" y1="31.75" x2="7.62" y2="27.94" width="0.2032" layer="1"/>
+<wire x1="7.62" y1="27.94" x2="7.2898" y2="27.6098" width="0.2032" layer="1"/>
 </signal>
 <signal name="SDI1">
@@
 <via x="89.2302" y="6.4008" extent="1-16" drill="0.35"/>
 <via x="95.7072" y="11.5824" extent="1-16" drill="0.35"/>
+<contactref element="IC3" pad="1"/>
+<wire x1="3.81" y1="28.194" x2="3.81" y2="28.8798" width="0.2032" layer="1"/>
+<wire x1="2.4384" y1="26.8224" x2="3.81" y2="28.194" width="0.2032" layer="1"/>
+<wire x1="2.4384" y1="15.0114" x2="2.4384" y2="26.8224" width="0.2032" layer="1"/>
+<wire x1="7.8486" y1="9.6012" x2="2.4384" y2="15.0114" width="0.2032" layer="1"/>
+<wire x1="7.8486" y1="7.6962" x2="7.8486" y2="9.6012" width="0.2032" layer="1"/>
+<wire x1="13.7922" y1="1.7526" x2="7.8486" y2="7.6962" width="0.2032" layer="1"/>
+<wire x1="86.0298" y1="1.7526" x2="13.7922" y2="1.7526" width="0.2032" layer="1"/>
+<wire x1="95.7072" y1="11.43" x2="86.0298" y2="1.7526" width="0.2032" layer="1"/>
+<wire x1="3.81" y1="28.8798" x2="3.88" y2="28.895" width="0.2032" layer="1"/>
+<wire x1="95.7072" y1="11.43" x2="95.7072" y2="11.5824" width="0.2032" layer="1"/>
+<contactref element="C27" pad="1"/>
+<wire x1="3.2766" y1="33.3756" x2="4.191" y2="34.29" width="0.2032" layer="16"/>
+<wire x1="3.2766" y1="29.4894" x2="3.2766" y2="33.3756" width="0.2032" layer="1"/>
+<wire x1="3.81" y1="28.956" x2="3.2766" y2="29.4894" width="0.2032" layer="1"/>
+<wire x1="4.191" y1="34.29" x2="4.23" y2="34.29" width="0.2032" layer="16"/>
+<wire x1="3.81" y1="28.956" x2="3.88" y2="28.895" width="0.2032" layer="1"/>
+<via x="3.2766" y="33.3756" extent="1-16" drill="0.35"/>
 </signal>
 <signal name="PGD">
@@
 <wire x1="95.25" y1="31.7754" x2="95.25" y2="31.75" width="0.1524" layer="2"/>
 </signal>
+<signal name="3.3REG" class="1">
+<contactref element="IC3" pad="2"/>
+<contactref element="AVDD_JUMPER" pad="1"/>
+<wire x1="3.8862" y1="27.7368" x2="3.8862" y2="27.051" width="0.2032" layer="1"/>
+<wire x1="5.0292" y1="28.8798" x2="3.8862" y2="27.7368" width="0.2032" layer="1"/>
+<wire x1="5.0292" y1="32.766" x2="5.0292" y2="28.8798" width="0.2032" layer="1"/>
+<wire x1="3.8862" y1="27.051" x2="3.88" y2="26.985" width="0.2032" layer="1"/>
+<wire x1="5.0292" y1="32.766" x2="5.08" y2="32.766" width="0.2032" layer="1"/>
+</signal>
+<signal name="AVDD_IN" class="1">
+<contactref element="E1" pad="1"/>
+<contactref element="AVDD_JUMPER" pad="2"/>
+<contactref element="C28" pad="1"/>
+<wire x1="4.2672" y1="26.1366" x2="4.2672" y2="20.3454" width="0.2032" layer="1"/>
+<wire x1="4.2672" y1="29.7942" x2="4.2672" y2="26.1366" width="0.2032" layer="2"/>
+<wire x1="4.2672" y1="31.7754" x2="4.2672" y2="29.7942" width="0.2032" layer="1"/>
+<wire x1="3.9624" y1="32.0802" x2="4.2672" y2="31.7754" width="0.2032" layer="1"/>
+<wire x1="3.9624" y1="33.4518" x2="3.9624" y2="32.0802" width="0.2032" layer="1"/>
+<wire x1="4.8006" y1="34.29" x2="3.9624" y2="33.4518" width="0.2032" layer="1"/>
+<wire x1="5.08" y1="34.29" x2="4.8006" y2="34.29" width="0.2032" layer="1"/>
+<wire x1="4.2672" y1="20.3454" x2="4.28" y2="20.32" width="0.2032" layer="1"/>
+<wire x1="2.8956" y1="13.716" x2="2.8956" y2="13.9446" width="0.2032" layer="16"/>
+<wire x1="2.1336" y1="12.954" x2="2.8956" y2="13.716" width="0.2032" layer="16"/>
+<wire x1="2.1336" y1="24.003" x2="2.1336" y2="12.954" width="0.2032" layer="15"/>
+<wire x1="4.2672" y1="26.1366" x2="2.1336" y2="24.003" width="0.2032" layer="15"/>
+<wire x1="2.8956" y1="13.9446" x2="2.96" y2="13.97" width="0.2032" layer="16"/>
+<via x="4.2672" y="26.1366" extent="1-16" drill="0.35"/>
+<via x="4.2672" y="29.7942" extent="1-16" drill="0.35"/>
+<via x="2.1336" y="12.954" extent="1-16" drill="0.35"/>
+</signal>
 </signals>

Commit message: max SPI2 speed
Parts:
- R11: value 100 ohm -> 50 ohm
Changed lines of the file:
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@@
 <attribute name="VALUE" x="109.22" y="8.89" size="0.0254" layer="27"/>
 </element>
-<element name="R11" library="rcl" library_urn="urn:adsk.eagle:library:334" package="R0805" package3d_urn="urn:adsk.eagle:package:23553/2" value="100 ohm" x="41.91" y="8.89" smashed="yes" rot="MR0">
+<element name="R11" library="rcl" library_urn="urn:adsk.eagle:library:334" package="R0805" package3d_urn="urn:adsk.eagle:package:23553/2" value="50 ohm" x="41.91" y="8.89" smashed="yes" rot="MR0">
 <attribute name="NAME" x="42.545" y="10.16" size="1.27" layer="26" rot="MR0"/>
 <attribute name="POPULARITY" value="85" x="41.91" y="8.89" size="1.778" layer="28" rot="MR0" display="off"/>

Commit message: up
Parts:
- added USBC-PWR: USBC-PWR, con-lstb:MA04-1
- R12, R13: value 100 ohm -> 50 ohm
- moved TP24 15.3 mm to (102.9, 22.9)
- moved SW2 1.27 mm to (109.2, 22.9)
- renumbered TP3 to TP3_VSS
Connections:
- net RA8: now also GLCD.9
- net RA9: now also GLCD.10
- net VIN_PWR: now also USBC-PWR.4
- net VSS: now also USBC-PWR.1
Routing:
- net RA9: track 136.6 -> 182.4 mm
- net RA8: track 129.0 -> 166.8 mm
- net VIN_PWR: track 14.1 -> 28.8 mm

Commit message: up
Parts:
- turned R4 to 270 degrees
Connections:
- net RA11 renamed TEST_P1
- removed net RA8: GLCD.9, PWM.8, U1.7
- removed net RA9: GLCD.10, PWM.9, U1.8
- removed net RB1: MISC_ANA.3, U1.21
- removed net RB5: MISC_ANA.4, U1.17
- new net RB1_DU: MISC_ANA.4, U1.21
- new net RC7: PWM.2, U1.36
- new net RC8: PWM.3, U1.35
- new net RD2: MISC_ANA.3, U1.53
- net DLED: now also U1.17; no longer U1.53
- net PWM1H: now also GLCD.10, PWM.9, U1.8; no longer PWM.3, U1.35
- net PWM1L: now also GLCD.9, PWM.8, U1.7; no longer PWM.2, U1.36
Routing:
- net RA9: track 182.4 -> 0.00 mm, vias 2 -> 0
- net RA8: track 166.8 -> 0.00 mm, vias 2 -> 0
- net RC8: track 0.00 -> 102.5 mm, vias 0 -> 4
- net RC7: track 0.00 -> 100.5 mm, vias 0 -> 2
- net PWM1H: track 102.5 -> 182.4 mm, vias 4 -> 2
- net RB1_DU: track 0.00 -> 70.9 mm, vias 0 -> 3
- net RB1: track 70.8 -> 0.00 mm, vias 3 -> 0
- net PWM1L: track 100.5 -> 166.8 mm
- net RB5: track 59.8 -> 0.00 mm, vias 2 -> 0
- net RD2: track 0.00 -> 37.8 mm, vias 0 -> 2
- net DLED: track 31.2 -> 66.8 mm, vias 0 -> 2
- net RLED: track 43.5 -> 27.1 mm
- net N$3: track 4.87 -> 2.52 mm

Commit message: finish V1.1 board
Parts:
- added C29: 0.1uf, rcl:C0603
- R11, R12, R13: device rcl:R0805 -> rcl:R0603
- moved R11 1.80 mm to (40.6, 7.62)
- moved R12 1.80 mm to (40.6, 14.0)
- moved R13 1.80 mm to (40.6, 11.4)
Connections:
- net RESET_SW: now also C29.1
- net SCK2: now also R13.2; no longer R13.1
- net SDI2: now also R11.2; no longer R11.1
- net SDO2: now also R12.2; no longer R12.1
- net VSS: now also C29.2, R11.1, R12.1, R13.1; no longer R11.2, R12.2, R13.2
Routing:
- net RESET_SW: track 55.2 -> 61.1 mm
- net SCK2: track 39.7 -> 34.5 mm
- net SDI2: track 32.5 -> 30.3 mm, vias 2 -> 3
- net SDO2: track 32.2 -> 31.1 mm
