File: pic32ak_fe.brd (EAGLE design)
At the start: 119.4 x 77.1 mm, 104 parts, among them IC1 NCP1117LPST33T3G, IC2 SFH6916, IC3 NCP51460SN33T1G, J1 CONBNC001, J2 CONBNC001, J3 CONBNC001, J4 CONBNC001, J5 5227222-3, SW1 PTS635SL50LFS, SW2 PTS635SL50LFS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

Commit message: up
Parts:
- added TEST_P1: PTR1PAD1-20, testpad:P1-20
Connections:
- net TEST_P1: now also TEST_P1.TP
Routing:
- net TEST_P1: track 132.9 -> 147.9 mm
Changed lines of the file:
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@@
 <attribute name="VALUE" x="71.755" y="8.255" size="1.27" layer="28" rot="MR0"/>
+</element>
+<element name="TEST_P1" library="testpad" library_urn="urn:adsk.eagle:library:385" package="P1-20" package3d_urn="urn:adsk.eagle:package:27950/1" value="PTR1PAD1-20" x="99.06" y="67.31" smashed="yes">
+<attribute name="NAME" x="94.996" y="69.088" size="1.27" layer="25" ratio="10"/>
+<attribute name="POPULARITY" value="3" x="99.06" y="67.31" size="1.778" layer="27" display="off"/>
+<attribute name="TP_SIGNAL_NAME" value="" x="99.06" y="67.31" size="1.778" layer="27" display="off"/>
+<attribute name="VALUE" x="99.06" y="67.31" size="0.0254" layer="27"/>
 </element>
 </elements>
@@
 <wire x1="79.7814" y1="20.3454" x2="80.8482" y2="21.4122" width="0.2032" layer="1"/>
 <wire x1="80.8482" y1="22.7838" x2="80.86" y2="22.86" width="0.2032" layer="1"/>
-<wire x1="79.7814" y1="20.3454" x2="79.7814" y2="20.32" width="0.2032" layer="1"/>
 <wire x1="61.5696" y1="5.0292" x2="60.96" y2="5.0292" width="0.2032" layer="15"/>
 <wire x1="63.246" y1="3.3528" x2="61.5696" y2="5.0292" width="0.2032" layer="15"/>
@@
 <wire x1="5.4102" y1="28.2702" x2="6.1722" y2="29.0322" width="0.2032" layer="1"/>
 <wire x1="5.4102" y1="21.5646" x2="5.4102" y2="28.2702" width="0.2032" layer="1"/>
+<wire x1="79.7814" y1="20.3454" x2="79.7814" y2="20.32" width="0.2032" layer="1"/>
 </signal>
 <signal name="VSS" class="1">
@@
 <via x="13.335" y="22.7076" extent="1-16" drill="0.35"/>
 <via x="10.4394" y="29.8704" extent="1-16" drill="0.35"/>
+<contactref element="TEST_P1" pad="TP"/>
+<wire x1="103.251" y1="67.3608" x2="99.06" y2="67.3608" width="0.1524" layer="1"/>
+<wire x1="104.6988" y1="68.8086" x2="103.251" y2="67.3608" width="0.1524" layer="1"/>
+<wire x1="112.014" y1="68.8086" x2="104.6988" y2="68.8086" width="0.1524" layer="1"/>
+<wire x1="113.0046" y1="69.7992" x2="112.014" y2="68.8086" width="0.1524" layer="1"/>
+<wire x1="99.06" y1="67.3608" x2="99.06" y2="67.31" width="0.1524" layer="1"/>
+<wire x1="113.0046" y1="69.7992" x2="113.03" y2="69.85" width="0.1524" layer="1"/>
 </signal>
 <signal name="PWM1L">
