File: pic32ak_fe.brd (EAGLE design)
At the start: 119.4 x 77.1 mm, 105 parts, among them IC1 NCP1117LPST33T3G, IC2 SFH6916, IC3 NCP51460SN33T1G, J1 CONBNC001, J2 CONBNC001, J3 CONBNC001, J4 CONBNC001, J5 5227222-3, SW1 PTS635SL50LFS, SW2 PTS635SL50LFS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

Commit message: up
Connections:
- net RB1_DU renamed RB1
Changed lines of the file:
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@@
 </element>
 <element name="C26" library="rcl" library_urn="urn:adsk.eagle:library:334" package="C0603" package3d_urn="urn:adsk.eagle:package:23616/2" value="0.1uf" x="80.01" y="22.86" smashed="yes" rot="R180">
-<attribute name="NAME" x="80.645" y="22.225" size="1.27" layer="25" rot="R180"/>
+<attribute name="NAME" x="78.105" y="24.765" size="1.27" layer="25" rot="R180"/>
 <attribute name="POPULARITY" value="37" x="80.01" y="22.86" size="1.778" layer="27" rot="R180" display="off"/>
 <attribute name="SPICEPREFIX" value="C" x="80.01" y="22.86" size="1.778" layer="27" rot="R180" display="off"/>
@@
 <wire x1="86.0298" y1="24.0792" x2="91.9734" y2="24.0792" width="0.1524" layer="15"/>
 </signal>
-<signal name="RB1_DU">
+<signal name="RB1">
 <contactref element="U1" pad="21"/>
 <wire x1="47.8536" y1="21.717" x2="56.2356" y2="21.717" width="0.1524" layer="1"/>

Commit message: up
Connections:
- net RC8 renamed RC6
Changed lines of the file:
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@@
 <wire x1="26.0604" y1="22.3266" x2="25.9969" y2="22.34" width="0.1524" layer="1"/>
 </signal>
-<signal name="RC8">
+<signal name="RC6">
 <contactref element="U1" pad="35"/>
 <contactref element="PWM" pad="3"/>

Commit message: up PCB
Parts:
- added EXT_SW: EXT_SW, pinhead:2X02
Connections:
- net SW1: now also EXT_SW.1
- net SW2: now also EXT_SW.2
- net VSS: now also EXT_SW.3, EXT_SW.4
Routing:
- net SW2: track 108.4 -> 116.8 mm
- net SW1: track 123.1 -> 128.4 mm
Other:
- board text added: "1"
Changed lines of the file:
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@@
 <hole x="3.81" y="73.66" drill="3.556"/>
 <hole x="115.57" y="73.66" drill="3.556"/>
+<text x="31.75" y="15.24" size="1.27" layer="16" font="vector" ratio="15" rot="MR0">1</text>
 </plain>
 <attributes>
@@
 <attribute name="TP_SIGNAL_NAME" value="" x="99.06" y="67.31" size="1.778" layer="27" display="off"/>
 <attribute name="VALUE" x="99.06" y="67.31" size="0.0254" layer="27"/>
+</element>
+<element name="EXT_SW" library="pinhead" library_urn="urn:adsk.eagle:library:325" package="2X02" package3d_urn="urn:adsk.eagle:package:22455/2" value="EXT_SW" x="102.87" y="33.02" smashed="yes" rot="R180">
+<attribute name="NAME" x="105.41" y="29.845" size="1.27" layer="25" ratio="10" rot="R180"/>
+<attribute name="POPULARITY" value="0" x="102.87" y="33.02" size="1.778" layer="27" rot="R180" display="off"/>
+<attribute name="VALUE" x="105.41" y="37.465" size="1.27" layer="27" rot="R180"/>
 </element>
 </elements>
@@
 <contactref element="R13" pad="1"/>
 <contactref element="C29" pad="2"/>
+<contactref element="EXT_SW" pad="3"/>
+<contactref element="EXT_SW" pad="4"/>
 </signal>
 <signal name="SDI1">
@@
 <wire x1="95.0976" y1="11.3538" x2="86.1822" y2="2.4384" width="0.1524" layer="1"/>
 <wire x1="95.0976" y1="18.2118" x2="95.0976" y2="11.3538" width="0.1524" layer="1"/>
-<wire x1="107.2134" y1="30.3276" x2="95.0976" y2="18.2118" width="0.1524" layer="1"/>
+<wire x1="107.2134" y1="30.3276" x2="107.1753" y2="30.2895" width="0.1524" layer="1"/>
+<wire x1="107.1753" y1="30.2895" x2="95.0976" y2="18.2118" width="0.1524" layer="1"/>
 <wire x1="109.1946" y1="30.3276" x2="107.2134" y2="30.3276" width="0.1524" layer="1"/>
 <wire x1="20.574" y1="27.2796" x2="20.57" y2="27.2669" width="0.1524" layer="1"/>
@@
 <via x="20.574" y="28.4988" extent="1-16" drill="0.35"/>
 <via x="56.3118" y="2.4384" extent="1-16" drill="0.35"/>
+<contactref element="EXT_SW" pad="1"/>
+<wire x1="104.1654" y1="33.2994" x2="104.1654" y2="34.29" width="0.1524" layer="1"/>
+<wire x1="107.1753" y1="30.2895" x2="104.1654" y2="33.2994" width="0.1524" layer="1"/>
+<wire x1="104.1654" y1="34.29" x2="104.14" y2="34.29" width="0.1524" layer="1"/>
 </signal>
 <signal name="SW2">
@@
 <via x="75.438" y="37.6428" extent="1-16" drill="0.35"/>
 <wire x1="107.5182" y1="16.4592" x2="109.1946" y2="16.4592" width="0.1524" layer="15"/>
-<wire x1="86.7156" y1="37.2618" x2="107.5182" y2="16.4592" width="0.1524" layer="15"/>
+<wire x1="86.7156" y1="37.2618" x2="98.1837" y2="25.7937" width="0.1524" layer="15"/>
+<wire x1="98.1837" y1="25.7937" x2="107.5182" y2="16.4592" width="0.1524" layer="15"/>
 <wire x1="86.7156" y1="37.6428" x2="86.7156" y2="37.2618" width="0.1524" layer="15"/>
 <wire x1="109.1946" y1="16.4592" x2="109.22" y2="16.36" width="0.1524" layer="15"/>
+<contactref element="EXT_SW" pad="2"/>
+<wire x1="98.1837" y1="25.7937" x2="104.14" y2="31.75" width="0.1524" layer="15"/>
 </signal>
 <signal name="TXDE">

Commit message: up
Parts:
- added BISS-C: BISS-C, con-lstb:MA10-1
- added BISS_DE1: BISS_DE1, jumper:SJ_2
- added BISS_DE2: BISS_DE2, jumper:SJ_2
- added C30: 0.1uf, rcl:C0603
- added C31: 1000pf, rcl:C0603
- added IC4: SN65C1168EPWR, SN65C1168EPWR:SOP65P640X120-16N
- added RS422_IN: PTR1PAD1-13, testpad:P1-13
Connections:
- new net MA+: BISS-C.6, IC4.13
- new net MA-: BISS-C.7, IC4.14
- new net MO+: BISS-C.4, IC4.11
- new net MO-: BISS-C.5, IC4.10
- new net N$11: BISS_DE1.2, IC4.4
- new net N$12: BISS_DE2.2, IC4.12
- new net N$19: IC4.5, RS422_IN.TP
- new net RS422_I+: BISS-C.2, IC4.7
- new net RS422_I-: BISS-C.3, IC4.6
- new net SL+: BISS-C.8, IC4.1
- new net SL-: BISS-C.9, IC4.2
- net RA6: now also IC4.9
- net RB1: now also IC4.15
- net RD2: now also IC4.3
- net VIN: now also BISS-C.10, BISS_DE1.3, BISS_DE2.1, C30.1, C31.1, IC4.16
- net VSS: now also BISS-C.1, BISS_DE1.1, BISS_DE2.3, C30.2, C31.2, IC4.8
Routing:
- net VIN: track 186.1 -> 315.3 mm, vias 3 -> 4
- net MA-: track 0.00 -> 63.9 mm, vias 0 -> 1
- net MA+: track 0.00 -> 57.6 mm, vias 0 -> 2
- net SL-: track 0.00 -> 56.7 mm, vias 0 -> 1
- net SL+: track 0.00 -> 53.2 mm, vias 0 -> 1
- net MO-: track 0.00 -> 52.5 mm, vias 0 -> 2
- net MO+: track 0.00 -> 49.3 mm, vias 0 -> 1
- net RS422_I-: track 0.00 -> 42.4 mm, vias 0 -> 2
- net RS422_I+: track 0.00 -> 41.9 mm, vias 0 -> 1
- net N$19: track 0.00 -> 30.6 mm, vias 0 -> 1
- net RA6: track 108.2 -> 133.9 mm, vias 0 -> 1
- net RB1: track 70.9 -> 94.2 mm, vias 3 -> 5
- net RD2: track 37.8 -> 59.7 mm, vias 2 -> 3
- net N$12: track 0.00 -> 18.5 mm
- net N$11: track 0.00 -> 4.84 mm

Commit message: up
Parts:
- added C32: 10uf, rcl:C0805
- added R14, R15, R16, R17: 120 ohm, rcl:R0603
Connections:
- net MA+: now also R15.2
- net MA-: now also R15.1
- net MO+: now also R16.2
- net MO-: now also R16.1
- net RS422_I+: now also R17.2
- net RS422_I-: now also R17.1
- net SL+: now also R14.2
- net SL-: now also R14.1
- net VIN: now also C32.1
- net VSS: now also C32.2
Routing:
- net RS422_I-: track 42.4 -> 47.4 mm, vias 2 -> 3
- net RS422_I+: track 41.9 -> 46.8 mm, vias 1 -> 2
- net MO+: track 49.3 -> 54.3 mm, vias 1 -> 2
- net MO-: track 52.5 -> 57.5 mm, vias 2 -> 3
- net SL+: track 53.2 -> 57.3 mm
- net MA-: track 63.9 -> 67.9 mm
- net SL-: track 56.7 -> 60.7 mm
- net MA+: track 57.6 -> 60.8 mm
- net VIN: track 315.3 -> 317.9 mm

Commit message: up
Parts:
- added D1: 5.6V, diode:SMB
Connections:
- net VIN: now also D1.C
- net VSS: now also D1.A
Routing:
- net VIN: track 317.9 -> 321.4 mm
Changed lines of the file:
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@@
 <layer number="97" name="Info" color="7" fill="1" visible="no" active="no"/>
 <layer number="98" name="Guide" color="6" fill="1" visible="no" active="no"/>
+<layer number="99" name="SpiceOrder" color="5" fill="1" visible="no" active="no"/>
 </layers>
 <board>
@@
 </class>
 <class number="1" name="current" width="0.2032" drill="0">
+</class>
+<class number="2" name="high_current" width="0.3048" drill="0">
 </class>
 </classes>
@@
 </element>
 <element name="FUSE" library="rcl" library_urn="urn:adsk.eagle:library:334" package="R0805" package3d_urn="urn:adsk.eagle:package:23553/2" value="0 ohm" x="97.79" y="12.7" smashed="yes">
-<attribute name="NAME" x="95.885" y="13.97" size="1.27" layer="25"/>
+<attribute name="NAME" x="100.965" y="12.7" size="1.27" layer="25"/>
 <attribute name="POPULARITY" value="85" x="97.79" y="12.7" size="1.778" layer="27" display="off"/>
 <attribute name="SPICEPREFIX" value="R" x="97.79" y="12.7" size="1.778" layer="27" display="off"/>
@@
 <attribute name="SPICEPREFIX" value="C" x="50.8" y="71.12" size="1.778" layer="28" rot="MR180" display="off"/>
 <attribute name="VALUE" x="49.53" y="73.66" size="1.27" layer="28" rot="MR180"/>
+</element>
+<element name="D1" library="diode" library_urn="urn:adsk.eagle:library:210" package="SMB" package3d_urn="urn:adsk.eagle:package:43404/2" value="5.6V" x="93.98" y="16.51" smashed="yes" rot="MR90">
+<attribute name="NAME" x="97.409" y="15.621" size="1.27" layer="26" rot="MR90"/>
+<attribute name="POPULARITY" value="11" x="93.98" y="16.51" size="1.778" layer="28" rot="MR90" display="off"/>
+<attribute name="VALUE" x="90.551" y="14.351" size="1.27" layer="28" rot="MR90"/>
 </element>
 </elements>
@@
 <contactref element="BISS-C" pad="1"/>
 <contactref element="C32" pad="2"/>
+<contactref element="D1" pad="A"/>
 </signal>
 <signal name="SDI1">
@@
 <wire x1="49.911" y1="71.0946" x2="49.85" y2="71.12" width="0.2032" layer="16"/>
 <wire x1="49.911" y1="68.6562" x2="49.95" y2="68.58" width="0.2032" layer="16"/>
+<contactref element="D1" pad="C"/>
+<wire x1="94.0308" y1="13.4874" x2="94.0308" y2="14.2494" width="0.2032" layer="16"/>
+<wire x1="95.7072" y1="11.811" x2="94.0308" y2="13.4874" width="0.2032" layer="16"/>
+<wire x1="95.7072" y1="11.5824" x2="95.7072" y2="11.811" width="0.2032" layer="16"/>
+<wire x1="94.0308" y1="14.2494" x2="93.98" y2="14.31" width="0.2032" layer="16"/>
 </signal>
 <signal name="PGD">
@@
 <wire x1="52.8828" y1="27.2034" x2="53.34" y2="26.67" width="0.1524" layer="1"/>
 </signal>
-<signal name="VIN_PWR" class="1">
+<signal name="VIN_PWR" class="2">
 <contactref element="VIN_5+" pad="2"/>
 <contactref element="FUSE" pad="2"/>
 <contactref element="TP8" pad="TP"/>
-<wire x1="98.679" y1="18.2118" x2="98.679" y2="12.7254" width="0.2032" layer="1"/>
-<wire x1="97.8408" y1="19.05" x2="98.679" y2="18.2118" width="0.2032" layer="1"/>
-<wire x1="98.679" y1="12.7254" x2="98.74" y2="12.7" width="0.2032" layer="1"/>
-<wire x1="97.8408" y1="19.05" x2="97.79" y2="19.05" width="0.2032" layer="1"/>
-<wire x1="96.5454" y1="10.5918" x2="96.5454" y2="8.1534" width="0.2032" layer="1"/>
-<wire x1="96.5454" y1="8.1534" x2="96.5454" y2="6.4008" width="0.2032" layer="1"/>
-<wire x1="98.6028" y1="12.6492" x2="96.5454" y2="10.5918" width="0.2032" layer="1"/>
-<wire x1="96.5454" y1="6.4008" x2="96.52" y2="6.35" width="0.2032" layer="1"/>
-<wire x1="98.6028" y1="12.6492" x2="98.74" y2="12.7" width="0.2032" layer="1"/>
 <contactref element="USBC-PWR" pad="4"/>
-<wire x1="110.109" y1="6.4008" x2="110.49" y2="6.4008" width="0.2032" layer="1"/>
-<wire x1="108.3564" y1="8.1534" x2="110.109" y2="6.4008" width="0.2032" layer="1"/>
-<wire x1="96.5454" y1="8.1534" x2="108.3564" y2="8.1534" width="0.2032" layer="1"/>
-<wire x1="110.49" y1="6.4008" x2="110.49" y2="6.35" width="0.2032" layer="1"/>
+<wire x1="98.679" y1="18.2118" x2="98.679" y2="12.7254" width="0.3048" layer="1"/>
+<wire x1="97.8408" y1="19.05" x2="98.679" y2="18.2118" width="0.3048" layer="1"/>
+<wire x1="98.679" y1="12.7254" x2="98.74" y2="12.7" width="0.3048" layer="1"/>
+<wire x1="97.8408" y1="19.05" x2="97.79" y2="19.05" width="0.3048" layer="1"/>
+<wire x1="96.5454" y1="10.4394" x2="96.5454" y2="6.4008" width="0.3048" layer="1"/>
+<wire x1="98.679" y1="12.573" x2="96.5454" y2="10.4394" width="0.3048" layer="1"/>
+<wire x1="96.5454" y1="6.4008" x2="96.52" y2="6.35" width="0.3048" layer="1"/>
+<wire x1="98.679" y1="12.573" x2="98.74" y2="12.7" width="0.3048" layer="1"/>
+<wire x1="110.1852" y1="6.4008" x2="110.49" y2="6.4008" width="0.3048" layer="1"/>
+<wire x1="104.013" y1="12.573" x2="110.1852" y2="6.4008" width="0.3048" layer="1"/>
+<wire x1="98.8314" y1="12.573" x2="104.013" y2="12.573" width="0.3048" layer="1"/>
+<wire x1="110.49" y1="6.4008" x2="110.49" y2="6.35" width="0.3048" layer="1"/>
+<wire x1="98.8314" y1="12.573" x2="98.74" y2="12.7" width="0.3048" layer="1"/>
 </signal>
 <signal name="OA2IN">

Commit message: up
Parts:
- added C33, C34: 0.1uf, rcl:C0603
Connections:
- net SW1: now also C33.1
- net SW2: now also C34.1
- net VSS: now also C33.2, C34.2
Routing:
- net SW1: track 128.4 -> 132.7 mm
- net SW2: track 116.8 -> 121.1 mm
Changed lines of the file:
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@@
 <attribute name="VALUE" x="90.551" y="14.351" size="1.27" layer="28" rot="MR90"/>
+</element>
+<element name="C33" library="rcl" library_urn="urn:adsk.eagle:library:334" package="C0603" package3d_urn="urn:adsk.eagle:package:23616/2" value="0.1uf" x="114.3" y="30.48" smashed="yes" rot="MR180">
+<attribute name="NAME" x="113.665" y="29.845" size="1.27" layer="26" rot="MR180"/>
+<attribute name="POPULARITY" value="37" x="114.3" y="30.48" size="1.778" layer="28" rot="MR180" display="off"/>
+<attribute name="SPICEPREFIX" value="C" x="114.3" y="30.48" size="1.778" layer="28" rot="MR180" display="off"/>
+<attribute name="VALUE" x="113.665" y="32.385" size="1.27" layer="28" rot="MR180"/>
+</element>
+<element name="C34" library="rcl" library_urn="urn:adsk.eagle:library:334" package="C0603" package3d_urn="urn:adsk.eagle:package:23616/2" value="0.1uf" x="114.3" y="16.51" smashed="yes" rot="MR180">
+<attribute name="NAME" x="113.665" y="15.875" size="1.27" layer="26" rot="MR180"/>
+<attribute name="POPULARITY" value="37" x="114.3" y="16.51" size="1.778" layer="28" rot="MR180" display="off"/>
+<attribute name="SPICEPREFIX" value="C" x="114.3" y="16.51" size="1.778" layer="28" rot="MR180" display="off"/>
+<attribute name="VALUE" x="113.665" y="18.415" size="1.27" layer="28" rot="MR180"/>
 </element>
 </elements>
@@
 <contactref element="C32" pad="2"/>
 <contactref element="D1" pad="A"/>
+<contactref element="C33" pad="2"/>
+<contactref element="C34" pad="2"/>
 </signal>
 <signal name="SDI1">
@@
 <wire x1="107.1753" y1="30.2895" x2="104.1654" y2="33.2994" width="0.1524" layer="1"/>
 <wire x1="104.1654" y1="34.29" x2="104.14" y2="34.29" width="0.1524" layer="1"/>
+<contactref element="C33" pad="1"/>
+<wire x1="109.347" y1="30.48" x2="113.45" y2="30.48" width="0.1524" layer="16"/>
+<wire x1="109.2708" y1="30.4038" x2="109.347" y2="30.48" width="0.1524" layer="16"/>
+<wire x1="109.2708" y1="30.4038" x2="109.22" y2="30.33" width="0.1524" layer="16"/>
 </signal>
 <signal name="SW2">
@@
 <contactref element="EXT_SW" pad="2"/>
 <wire x1="98.1837" y1="25.7937" x2="104.14" y2="31.75" width="0.1524" layer="15"/>
+<contactref element="C34" pad="1"/>
+<wire x1="109.347" y1="16.4592" x2="113.3856" y2="16.4592" width="0.1524" layer="16"/>
+<wire x1="109.2708" y1="16.383" x2="109.347" y2="16.4592" width="0.1524" layer="16"/>
+<wire x1="113.3856" y1="16.4592" x2="113.45" y2="16.51" width="0.1524" layer="16"/>
+<wire x1="109.2708" y1="16.383" x2="109.22" y2="16.36" width="0.1524" layer="16"/>
 </signal>
 <signal name="TXDE">

Commit message: up
Parts:
- R1: value 100 ohm -> 56 ohm
- R11: value 50 ohm -> 120 ohm
- R3, R4, R5, R6: value 1K ohm -> 2.2K ohm
Changed lines of the file:
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@@
 <attribute name="VALUE" x="28.575" y="10.795" size="1.27" layer="28" rot="MR180"/>
 </element>
-<element name="R1" library="rcl" library_urn="urn:adsk.eagle:library:334" package="R0805" package3d_urn="urn:adsk.eagle:package:23553/2" value="100 ohm" x="38.1" y="29.21" smashed="yes" rot="MR0">
+<element name="R1" library="rcl" library_urn="urn:adsk.eagle:library:334" package="R0805" package3d_urn="urn:adsk.eagle:package:23553/2" value="56 ohm" x="38.1" y="29.21" smashed="yes" rot="MR0">
 <attribute name="NAME" x="42.545" y="29.21" size="1.27" layer="26" rot="MR0"/>
 <attribute name="POPULARITY" value="85" x="38.1" y="29.21" size="1.778" layer="28" rot="MR0" display="off"/>
@@
 <attribute name="VALUE" x="74.295" y="5.08" size="1.27" layer="28" rot="MR270"/>
 </element>
-<element name="R3" library="rcl" library_urn="urn:adsk.eagle:library:334" package="R0805" package3d_urn="urn:adsk.eagle:package:23553/2" value="1K ohm" x="45.72" y="31.75" smashed="yes" rot="R270">
+<element name="R3" library="rcl" library_urn="urn:adsk.eagle:library:334" package="R0805" package3d_urn="urn:adsk.eagle:package:23553/2" value="2.2K ohm" x="45.72" y="31.75" smashed="yes" rot="R270">
 <attribute name="NAME" x="46.99" y="28.575" size="1.27" layer="25" rot="R270"/>
 <attribute name="POPULARITY" value="85" x="45.72" y="31.75" size="1.778" layer="27" rot="R270" display="off"/>
@@
 <attribute name="VALUE" x="55.245" y="34.925" size="1.27" layer="27" rot="R90"/>
 </element>
-<element name="R4" library="rcl" library_urn="urn:adsk.eagle:library:334" package="R0805" package3d_urn="urn:adsk.eagle:package:23553/2" value="1K ohm" x="48.26" y="31.75" smashed="yes" rot="R270">
+<element name="R4" library="rcl" library_urn="urn:adsk.eagle:library:334" package="R0805" package3d_urn="urn:adsk.eagle:package:23553/2" value="2.2K ohm" x="48.26" y="31.75" smashed="yes" rot="R270">
 <attribute name="NAME" x="50.8" y="37.465" size="1.27" layer="25" rot="R270"/>
 <attribute name="POPULARITY" value="85" x="48.26" y="31.75" size="1.778" layer="27" rot="R270" display="off"/>
@@
 <attribute name="VALUE" x="45.72" y="32.385" size="1.27" layer="27" rot="R270"/>
 </element>
-<element name="R5" library="rcl" library_urn="urn:adsk.eagle:library:334" package="R0805" package3d_urn="urn:adsk.eagle:package:23553/2" value="1K ohm" x="50.8" y="31.75" smashed="yes" rot="R270">
+<element name="R5" library="rcl" library_urn="urn:adsk.eagle:library:334" package="R0805" package3d_urn="urn:adsk.eagle:package:23553/2" value="2.2K ohm" x="50.8" y="31.75" smashed="yes" rot="R270">
 <attribute name="NAME" x="49.53" y="28.575" size="1.27" layer="25" rot="R270"/>
 <attribute name="POPULARITY" value="85" x="50.8" y="31.75" size="1.778" layer="27" rot="R270" display="off"/>
@@
 <attribute name="VALUE" x="48.26" y="32.385" size="1.27" layer="27" rot="R270"/>
 </element>
-<element name="R6" library="rcl" library_urn="urn:adsk.eagle:library:334" package="R0805" package3d_urn="urn:adsk.eagle:package:23553/2" value="1K ohm" x="53.34" y="31.75" smashed="yes" rot="R270">
+<element name="R6" library="rcl" library_urn="urn:adsk.eagle:library:334" package="R0805" package3d_urn="urn:adsk.eagle:package:23553/2" value="2.2K ohm" x="53.34" y="31.75" smashed="yes" rot="R270">
 <attribute name="NAME" x="55.245" y="30.48" size="1.27" layer="25"/>
 <attribute name="POPULARITY" value="85" x="53.34" y="31.75" size="1.778" layer="27" rot="R270" display="off"/>
@@
 <attribute name="VALUE" x="107.315" y="8.001" size="1.27" layer="27" ratio="10"/>
 </element>
-<element name="R11" library="rcl" library_urn="urn:adsk.eagle:library:334" package="R0603" package3d_urn="urn:adsk.eagle:package:23555/3" value="50 ohm" x="40.64" y="7.62" smashed="yes" rot="MR0">
+<element name="R11" library="rcl" library_urn="urn:adsk.eagle:library:334" package="R0603" package3d_urn="urn:adsk.eagle:package:23555/3" value="120 ohm" x="40.64" y="7.62" smashed="yes" rot="MR0">
 <attribute name="NAME" x="45.085" y="6.985" size="1.27" layer="26" rot="MR0"/>
 <attribute name="POPULARITY" value="77" x="40.64" y="7.62" size="1.778" layer="28" rot="MR0" display="off"/>
