File: pic32ak_fe.sch (EAGLE design)
At the start: 68 parts, among them IC1 NCP1117LPST33T3G, J1 CONBNC001, J2 CONBNC001, J3 CONBNC001, J4 CONBNC001, J5 22-27-2021-02, U1 PIC32AK1216GC41064-E/PT, U2 IS66WVS4M8BLL-104NLI, X1 22-23-2021, Y1 KC2520Z8.00000C1KX00

Commit message: up
Parts:
- removed TP7, TP8: PTR1PAD1-20, testpad:PTR1PAD1-20
Connections:
- net DLED: no longer TP8.TP
- net RLED: no longer TP7.TP
Changed lines of the file:
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@@
 <part name="TP5" library="testpad" library_urn="urn:adsk.eagle:library:385" deviceset="PTR1" device="PAD1-13" package3d_urn="urn:adsk.eagle:package:27946/1"/>
 <part name="TP6" library="testpad" library_urn="urn:adsk.eagle:library:385" deviceset="PTR1" device="PAD1-13" package3d_urn="urn:adsk.eagle:package:27946/1"/>
-<part name="TP7" library="testpad" library_urn="urn:adsk.eagle:library:385" deviceset="PTR1" device="PAD1-20" package3d_urn="urn:adsk.eagle:package:27950/1"/>
-<part name="TP8" library="testpad" library_urn="urn:adsk.eagle:library:385" deviceset="PTR1" device="PAD1-20" package3d_urn="urn:adsk.eagle:package:27950/1"/>
 <part name="TP9" library="testpad" library_urn="urn:adsk.eagle:library:385" deviceset="PTR1" device="PAD1-20" package3d_urn="urn:adsk.eagle:package:27950/1"/>
 <part name="TP10" library="testpad" library_urn="urn:adsk.eagle:library:385" deviceset="PTR1" device="PAD1-20" package3d_urn="urn:adsk.eagle:package:27950/1"/>
@@
 <attribute name="NAME" x="224.79" y="87.884" size="1.778" layer="95" rot="R180"/>
 <attribute name="TP_SIGNAL_NAME" x="220.98" y="90.17" size="1.778" layer="97" rot="R90"/>
-</instance>
-<instance part="TP7" gate="G$1" x="241.3" y="111.76" smashed="yes" rot="R180">
-<attribute name="NAME" x="242.316" y="118.11" size="1.778" layer="95" rot="R270"/>
-<attribute name="TP_SIGNAL_NAME" x="240.03" y="114.3" size="1.778" layer="97" rot="R180"/>
-</instance>
-<instance part="TP8" gate="G$1" x="248.92" y="111.76" smashed="yes" rot="R180">
-<attribute name="NAME" x="249.936" y="118.11" size="1.778" layer="95" rot="R270"/>
-<attribute name="TP_SIGNAL_NAME" x="247.65" y="114.3" size="1.778" layer="97" rot="R180"/>
 </instance>
 <instance part="TP9" gate="G$1" x="256.54" y="111.76" smashed="yes" rot="R180">
@@
 <pinref part="R4" gate="G$1" pin="2"/>
 <junction x="241.3" y="93.98"/>
+<label x="241.3" y="101.6" size="1.778" layer="95" rot="R90"/>
 <junction x="241.3" y="109.22"/>
-<label x="241.3" y="101.6" size="1.778" layer="95" rot="R90"/>
-<pinref part="TP7" gate="G$1" pin="TP"/>
 </segment>
 </net>
@@
 <pinref part="R5" gate="G$1" pin="2"/>
 <junction x="248.92" y="93.98"/>
+<label x="248.92" y="101.6" size="1.778" layer="95" rot="R90"/>
 <junction x="248.92" y="109.22"/>
-<label x="248.92" y="101.6" size="1.778" layer="95" rot="R90"/>
-<pinref part="TP8" gate="G$1" pin="TP"/>
-</segment>
-</net>
+</segment>
+</net>

Commit message: up
Parts:
- renumbered J5 to R_RESET, TP9 to TEST_P0, X1 to VIN_5+
Changed lines of the file:
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@@
 <part name="R6" library="rcl" library_urn="urn:adsk.eagle:library:334" deviceset="R-US_" device="R0805" package3d_urn="urn:adsk.eagle:package:23553/2" value="1K ohm"/>
 <part name="MISC_ANA" library="pinhead" library_urn="urn:adsk.eagle:library:325" deviceset="PINHD-1X6" device="/90" package3d_urn="urn:adsk.eagle:package:22475/2" value="MISC_ANA"/>
-<part name="X1" library="con-molex" library_urn="urn:adsk.eagle:library:165" deviceset="22-23-2021" device="" package3d_urn="urn:adsk.eagle:package:8078633/1"/>
+<part name="VIN_5+" library="con-molex" library_urn="urn:adsk.eagle:library:165" deviceset="22-23-2021" device="" package3d_urn="urn:adsk.eagle:package:8078633/1"/>
 <part name="VSS20" library="supply1" library_urn="urn:adsk.eagle:library:371" deviceset="VSS" device=""/>
 <part name="FUSE" library="rcl" library_urn="urn:adsk.eagle:library:334" deviceset="R-US_" device="R0805" package3d_urn="urn:adsk.eagle:package:23553/2" value="0 ohm"/>
@@
 <part name="TP5" library="testpad" library_urn="urn:adsk.eagle:library:385" deviceset="PTR1" device="PAD1-13" package3d_urn="urn:adsk.eagle:package:27946/1"/>
 <part name="TP6" library="testpad" library_urn="urn:adsk.eagle:library:385" deviceset="PTR1" device="PAD1-13" package3d_urn="urn:adsk.eagle:package:27946/1"/>
-<part name="TP9" library="testpad" library_urn="urn:adsk.eagle:library:385" deviceset="PTR1" device="PAD1-20" package3d_urn="urn:adsk.eagle:package:27950/1"/>
+<part name="TEST_P0" library="testpad" library_urn="urn:adsk.eagle:library:385" deviceset="PTR1" device="PAD1-20" package3d_urn="urn:adsk.eagle:package:27950/1"/>
 <part name="TP10" library="testpad" library_urn="urn:adsk.eagle:library:385" deviceset="PTR1" device="PAD1-20" package3d_urn="urn:adsk.eagle:package:27950/1"/>
 <part name="TP11" library="testpad" library_urn="urn:adsk.eagle:library:385" deviceset="PTR1" device="PAD1-20" package3d_urn="urn:adsk.eagle:package:27950/1"/>
 <part name="TP12" library="testpad" library_urn="urn:adsk.eagle:library:385" deviceset="PTR1" device="PAD1-20" package3d_urn="urn:adsk.eagle:package:27950/1"/>
-<part name="J5" library="con-molex" library_urn="urn:adsk.eagle:library:165" deviceset="22-?-02" device="27-2021" package3d_urn="urn:adsk.eagle:package:8078645/1"/>
+<part name="R_RESET" library="con-molex" library_urn="urn:adsk.eagle:library:165" deviceset="22-?-02" device="27-2021" package3d_urn="urn:adsk.eagle:package:8078645/1"/>
 <part name="VSS27" library="supply1" library_urn="urn:adsk.eagle:library:371" deviceset="VSS" device=""/>
 <part name="TP13" library="testpad" library_urn="urn:adsk.eagle:library:385" deviceset="PTR1" device="PAD1-13" package3d_urn="urn:adsk.eagle:package:27946/1"/>
@@
 <attribute name="VALUE" x="26.67" y="68.58" size="1.778" layer="96" rot="R180"/>
 </instance>
-<instance part="X1" gate="-1" x="63.5" y="-88.9" smashed="yes" rot="R180">
+<instance part="VIN_5+" gate="-1" x="63.5" y="-88.9" smashed="yes" rot="R180">
 <attribute name="NAME" x="60.96" y="-88.138" size="1.524" layer="95" rot="R180"/>
 <attribute name="VALUE" x="64.262" y="-90.297" size="1.778" layer="96" rot="R180"/>
 </instance>
-<instance part="X1" gate="-2" x="63.5" y="-86.36" smashed="yes" rot="R180">
+<instance part="VIN_5+" gate="-2" x="63.5" y="-86.36" smashed="yes" rot="R180">
 <attribute name="NAME" x="60.96" y="-85.598" size="1.524" layer="95" rot="R180"/>
 </instance>
@@
 <attribute name="TP_SIGNAL_NAME" x="220.98" y="90.17" size="1.778" layer="97" rot="R90"/>
 </instance>
-<instance part="TP9" gate="G$1" x="256.54" y="111.76" smashed="yes" rot="R180">
+<instance part="TEST_P0" gate="G$1" x="256.54" y="111.76" smashed="yes" rot="R180">
 <attribute name="NAME" x="257.556" y="118.11" size="1.778" layer="95" rot="R270"/>
 <attribute name="TP_SIGNAL_NAME" x="255.27" y="114.3" size="1.778" layer="97" rot="R180"/>
@@
 <attribute name="TP_SIGNAL_NAME" x="285.75" y="68.58" size="1.778" layer="97" rot="R180"/>
 </instance>
-<instance part="J5" gate="-1" x="340.36" y="58.42" smashed="yes">
+<instance part="R_RESET" gate="-1" x="340.36" y="58.42" smashed="yes">
 <attribute name="NAME" x="342.9" y="57.658" size="1.524" layer="95"/>
 <attribute name="VALUE" x="339.598" y="59.817" size="1.778" layer="96"/>
 </instance>
-<instance part="J5" gate="-2" x="340.36" y="53.34" smashed="yes">
+<instance part="R_RESET" gate="-2" x="340.36" y="53.34" smashed="yes">
 <attribute name="NAME" x="342.9" y="52.578" size="1.524" layer="95"/>
 </instance>
@@
 </segment>
 <segment>
-<pinref part="X1" gate="-1" pin="S"/>
+<pinref part="VIN_5+" gate="-1" pin="S"/>
 <pinref part="VSS20" gate="G$1" pin="VSS"/>
 <junction x="66.04" y="-88.9"/>
@@
 </segment>
 <segment>
-<pinref part="J5" gate="-1" pin="S"/>
+<pinref part="R_RESET" gate="-1" pin="S"/>
 <pinref part="VSS27" gate="G$1" pin="VSS"/>
 <junction x="337.82" y="58.42"/>
@@
 <segment>
 <wire x1="320.04" y1="53.34" x2="337.82" y2="53.34" width="0.1524" layer="91"/>
-<pinref part="J5" gate="-2" pin="S"/>
+<pinref part="R_RESET" gate="-2" pin="S"/>
 <junction x="337.82" y="53.34"/>
 <junction x="320.04" y="53.34"/>
@@
 <junction x="256.54" y="93.98"/>
 <label x="256.54" y="101.6" size="1.778" layer="95" rot="R90"/>
-<pinref part="TP9" gate="G$1" pin="TP"/>
+<pinref part="TEST_P0" gate="G$1" pin="TP"/>
 </segment>
 </net>
 <net name="VIN_PWR" class="1">
 <segment>
-<pinref part="X1" gate="-2" pin="S"/>
+<pinref part="VIN_5+" gate="-2" pin="S"/>
 <wire x1="66.04" y1="-86.36" x2="73.66" y2="-86.36" width="0.1524" layer="91"/>
 <pinref part="FUSE" gate="G$1" pin="2"/>

Commit message: up
Parts:
- added J5: 5227222-3, 5227222-3:5227222-3
Connections:
- net PGC_DAC: now also J5.1
- net VSS: now also J5.2
Changed lines of the file:
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@@
 <part name="TP18" library="testpad" library_urn="urn:adsk.eagle:library:385" deviceset="PTR1" device="PAD1-13" package3d_urn="urn:adsk.eagle:package:27946/1"/>
 <part name="VSS28" library="supply1" library_urn="urn:adsk.eagle:library:371" deviceset="VSS" device=""/>
+<part name="J5" library="5227222-3" deviceset="5227222-3" device=""/>
 </parts>
 <sheets>
@@
 <instance part="VSS28" gate="G$1" x="210.82" y="-53.34" smashed="yes">
 <attribute name="VALUE" x="218.44" y="-53.34" size="1.778" layer="96" rot="R180"/>
+</instance>
+<instance part="J5" gate="G$1" x="60.96" y="60.96" smashed="yes">
+<attribute name="NAME" x="77.47" y="68.58" size="1.778" layer="95" align="center-left"/>
+<attribute name="VALUE" x="77.47" y="66.04" size="1.778" layer="96" align="center-left"/>
 </instance>
 </instances>
@@
 <junction x="210.82" y="-50.8"/>
 </segment>
+<segment>
+<wire x1="48.26" y1="60.96" x2="60.96" y2="60.96" width="0.1524" layer="91"/>
+<pinref part="J5" gate="G$1" pin="2"/>
+<junction x="60.96" y="60.96"/>
+<junction x="48.26" y="60.96"/>
+<label x="50.8" y="60.96" size="1.778" layer="95"/>
+</segment>
 </net>
 <net name="SDI1" class="0">
@@
 <label x="38.1" y="53.34" size="1.778" layer="95"/>
 </segment>
-</net>
+<segment>
+<wire x1="60.96" y1="58.42" x2="48.26" y2="58.42" width="0.1524" layer="91"/>
+<pinref part="J5" gate="G$1" pin="1"/>
+<junction x="60.96" y="58.42"/>
+<junction x="48.26" y="58.42"/>
+<label x="50.8" y="58.42" size="1.778" layer="95"/>
+</segment>
+</net>

Commit message: up
Parts:
- added ENCODER: Encoder, pinhead:PINHD-1X6/90
- added SJ1: QEI Voltage, jumper:SJ2W
- added TP7, TP8: PTR1PAD1-13, testpad:PTR1PAD1-13
Connections:
- new net QEI_A: ENCODER.2, U1.RP43/IOMD9/IOMF9/RC10
- new net QEI_B: ENCODER.3, U1.RP44/IOMD8/IOMF8/RC11
- new net QEI_H: ENCODER.5, U1.PGD3/RP36/PWM3H/IOMD0/RC3
- new net QEI_I: ENCODER.4, U1.RP37/PWM3L/IOMD1/RC4
- new net QEI_PWR: ENCODER.6, SJ1.2
- net VDD: now also SJ1.1
- net VIN: now also SJ1.3, TP7.TP
- net VIN_PWR: now also TP8.TP
- net VSS: now also ENCODER.1
Changed lines of the file:
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@@
 <part name="VSS28" library="supply1" library_urn="urn:adsk.eagle:library:371" deviceset="VSS" device=""/>
 <part name="J5" library="5227222-3" deviceset="5227222-3" device=""/>
+<part name="TP7" library="testpad" library_urn="urn:adsk.eagle:library:385" deviceset="PTR1" device="PAD1-13" package3d_urn="urn:adsk.eagle:package:27946/1"/>
+<part name="TP8" library="testpad" library_urn="urn:adsk.eagle:library:385" deviceset="PTR1" device="PAD1-13" package3d_urn="urn:adsk.eagle:package:27946/1"/>
+<part name="SJ1" library="jumper" library_urn="urn:adsk.eagle:library:252" deviceset="SJ2W" device="" package3d_urn="urn:adsk.eagle:package:15474/1" value="QEI Voltage"/>
+<part name="ENCODER" library="pinhead" library_urn="urn:adsk.eagle:library:325" deviceset="PINHD-1X6" device="/90" package3d_urn="urn:adsk.eagle:package:22475/2" value="Encoder"/>
+<part name="VDD12" library="supply1" library_urn="urn:adsk.eagle:library:371" deviceset="VDD" device=""/>
+<part name="VSS29" library="supply1" library_urn="urn:adsk.eagle:library:371" deviceset="VSS" device=""/>
 </parts>
 <sheets>
@@
 <attribute name="NAME" x="77.47" y="68.58" size="1.778" layer="95" align="center-left"/>
 <attribute name="VALUE" x="77.47" y="66.04" size="1.778" layer="96" align="center-left"/>
+</instance>
+<instance part="TP7" gate="G$1" x="91.44" y="-86.36" smashed="yes" rot="R90">
+<attribute name="NAME" x="105.41" y="-84.836" size="1.778" layer="95" rot="R180"/>
+<attribute name="TP_SIGNAL_NAME" x="93.98" y="-85.09" size="1.778" layer="97" rot="R90"/>
+</instance>
+<instance part="TP8" gate="G$1" x="76.2" y="-91.44" smashed="yes" rot="R90">
+<attribute name="NAME" x="90.17" y="-89.916" size="1.778" layer="95" rot="R180"/>
+<attribute name="TP_SIGNAL_NAME" x="78.74" y="-90.17" size="1.778" layer="97" rot="R90"/>
+</instance>
+<instance part="SJ1" gate="G$1" x="358.14" y="91.44" smashed="yes">
+<attribute name="NAME" x="360.68" y="91.821" size="1.778" layer="95"/>
+<attribute name="VALUE" x="360.68" y="89.535" size="1.778" layer="96"/>
+</instance>
+<instance part="ENCODER" gate="A" x="340.36" y="78.74" smashed="yes" rot="R180">
+<attribute name="NAME" x="346.71" y="67.945" size="1.778" layer="95" rot="R180"/>
+<attribute name="VALUE" x="346.71" y="88.9" size="1.778" layer="96" rot="R180"/>
+</instance>
+<instance part="VDD12" gate="G$1" x="358.14" y="99.06" smashed="yes">
+<attribute name="VALUE" x="365.76" y="99.06" size="1.778" layer="96" rot="R180"/>
+</instance>
+<instance part="VSS29" gate="G$1" x="342.9" y="68.58" smashed="yes">
+<attribute name="VALUE" x="365.76" y="71.12" size="1.778" layer="96" rot="R180"/>
 </instance>
 </instances>
@@
 <pinref part="VDD11" gate="G$1" pin="VDD"/>
 <junction x="210.82" y="-68.58"/>
+</segment>
+<segment>
+<pinref part="SJ1" gate="G$1" pin="1"/>
+<pinref part="VDD12" gate="G$1" pin="VDD"/>
+<junction x="358.14" y="96.52"/>
 </segment>
 </net>
@@
 <label x="50.8" y="60.96" size="1.778" layer="95"/>
 </segment>
+<segment>
+<pinref part="ENCODER" gate="A" pin="1"/>
+<pinref part="VSS29" gate="G$1" pin="VSS"/>
+<junction x="342.9" y="71.12"/>
+</segment>
 </net>
 <net name="SDI1" class="0">
@@
 <junction x="88.9" y="-86.36"/>
 <label x="86.36" y="-83.82" size="1.778" layer="95"/>
+<pinref part="TP7" gate="G$1" pin="TP"/>
+</segment>
+<segment>
+<wire x1="363.22" y1="86.36" x2="358.14" y2="86.36" width="0.1524" layer="91"/>
+<pinref part="SJ1" gate="G$1" pin="3"/>
+<junction x="358.14" y="86.36"/>
+<junction x="363.22" y="86.36"/>
+<label x="365.76" y="86.36" size="1.778" layer="95"/>
 </segment>
 </net>
@@
 <junction x="66.04" y="-86.36"/>
 <junction x="73.66" y="-86.36"/>
+<pinref part="TP8" gate="G$1" pin="TP"/>
+<wire x1="73.66" y1="-91.44" x2="73.66" y2="-86.36" width="0.1524" layer="91"/>
+<junction x="73.66" y="-91.44"/>
 </segment>
 </net>
@@
 </segment>
 </net>
+<net name="QEI_H" class="0">
+<segment>
+<pinref part="U1" gate="A" pin="PGD3/RP36/PWM3H/IOMD0/RC3"/>
+<wire x1="294.64" y1="-7.62" x2="309.88" y2="-7.62" width="0.1524" layer="91"/>
+<junction x="294.64" y="-7.62"/>
+<junction x="309.88" y="-7.62"/>
+<label x="317.5" y="-7.62" size="1.778" layer="95"/>
+</segment>
+<segment>
+<wire x1="342.9" y1="81.28" x2="358.14" y2="81.28" width="0.1524" layer="91"/>
+<pinref part="ENCODER" gate="A" pin="5"/>
+<junction x="342.9" y="81.28"/>
+<junction x="358.14" y="81.28"/>
+<label x="360.68" y="81.28" size="1.778" layer="95"/>
+</segment>
+</net>
+<net name="QEI_I" class="0">
+<segment>
+<pinref part="U1" gate="A" pin="RP37/PWM3L/IOMD1/RC4"/>
+<wire x1="294.64" y1="-5.08" x2="309.88" y2="-5.08" width="0.1524" layer="91"/>
+<junction x="294.64" y="-5.08"/>
+<junction x="309.88" y="-5.08"/>
+<label x="317.5" y="-5.08" size="1.778" layer="95"/>
+</segment>
+<segment>
+<wire x1="342.9" y1="78.74" x2="358.14" y2="78.74" width="0.1524" layer="91"/>
+<pinref part="ENCODER" gate="A" pin="4"/>
+<junction x="342.9" y="78.74"/>
+<junction x="358.14" y="78.74"/>
+<label x="360.68" y="78.74" size="1.778" layer="95"/>
+</segment>
+</net>
+<net name="QEI_B" class="0">
+<segment>
+<pinref part="U1" gate="A" pin="RP44/IOMD8/IOMF8/RC11"/>
+<wire x1="294.64" y1="0" x2="309.88" y2="0" width="0.1524" layer="91"/>
+<junction x="294.64" y="0"/>
+<junction x="309.88" y="0"/>
+<label x="317.5" y="0" size="1.778" layer="95"/>
+</segment>
+<segment>
+<wire x1="342.9" y1="76.2" x2="358.14" y2="76.2" width="0.1524" layer="91"/>
+<pinref part="ENCODER" gate="A" pin="3"/>
+<junction x="342.9" y="76.2"/>
+<junction x="358.14" y="76.2"/>
+<label x="360.68" y="76.2" size="1.778" layer="95"/>
+</segment>
+</net>
+<net name="QEI_A" class="0">
+<segment>
+<pinref part="U1" gate="A" pin="RP43/IOMD9/IOMF9/RC10"/>
+<wire x1="294.64" y1="-2.54" x2="309.88" y2="-2.54" width="0.1524" layer="91"/>
+<junction x="294.64" y="-2.54"/>
+<junction x="309.88" y="-2.54"/>
+<label x="317.5" y="-2.54" size="1.778" layer="95"/>
+</segment>
+<segment>
+<wire x1="342.9" y1="73.66" x2="358.14" y2="73.66" width="0.1524" layer="91"/>
+<pinref part="ENCODER" gate="A" pin="2"/>
+<junction x="342.9" y="73.66"/>
+<junction x="358.14" y="73.66"/>
+<label x="360.68" y="73.66" size="1.778" layer="95"/>
+</segment>
+</net>
+<net name="QEI_PWR" class="1">
+<segment>
+<pinref part="ENCODER" gate="A" pin="6"/>
+<pinref part="SJ1" gate="G$1" pin="2"/>
+<wire x1="342.9" y1="83.82" x2="353.06" y2="83.82" width="0.1524" layer="91"/>
+<wire x1="353.06" y1="83.82" x2="353.06" y2="91.44" width="0.1524" layer="91"/>
+<junction x="342.9" y="83.82"/>
+<junction x="353.06" y="91.44"/>
+<label x="340.36" y="91.44" size="1.778" layer="95"/>
+</segment>
+</net>

Commit message: up
Parts:
- added AC1: SCA3300-D01-1, SCA3300-D01-1:SCA3300-D01-1
- added C21, C22, C24: 0.1uf, rcl:C-USC0603
- added C23: 1000pf, rcl:C-USC0603
- added C25: 10uf, rcl:C-USC0805
Connections:
- new net IMU_CS: AC1.CSB, U1.PGD1/AD1AN5/CMP1C/ISRC0/IBIAS0/RP20/SDA1/RB3
- new net N$1: AC1.A_EXTC, C22.1
- new net N$6: AC1.D_EXTC, C21.1
- new net SCK3: AC1.SCK, U1.TMS/OA2IN-/AD1AN4/AD2ANN1/RP18/RB1
- new net SDI3: AC1.MISO, U1.AD1AN11/RP25/RB8
- new net SDO3: AC1.MOSI, U1.AD2AN10/RP26/RB9
- net VDD: now also AC1.DVIO, AC1.VDD, C23.1, C24.2, C25.2
- net VSS: now also AC1.AVSS, AC1.DVSS, AC1.EMC_GND, AC1.REERVED, C21.2, C22.2, C23.2, C24.1, C25.1

Commit message: up
Parts:
- added C26: 0.1uf, rcl:C-USC0603
Connections:
- net VDD: now also C26.1
- net VSS: now also C26.2
Changed lines of the file:
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@@
 <part name="VDD13" library="supply1" library_urn="urn:adsk.eagle:library:371" deviceset="VDD" device=""/>
 <part name="VSS32" library="supply1" library_urn="urn:adsk.eagle:library:371" deviceset="VSS" device=""/>
+<part name="C26" library="rcl" library_urn="urn:adsk.eagle:library:334" deviceset="C-US" device="C0603" package3d_urn="urn:adsk.eagle:package:23616/2" value="0.1uf"/>
+<part name="VSS33" library="supply1" library_urn="urn:adsk.eagle:library:371" deviceset="VSS" device=""/>
 </parts>
 <sheets>
@@
 <instance part="VSS32" gate="G$1" x="368.3" y="-101.6" smashed="yes">
 <attribute name="VALUE" x="375.92" y="-101.6" size="1.778" layer="96" rot="R180"/>
+</instance>
+<instance part="C26" gate="G$1" x="350.52" y="-86.36" smashed="yes" rot="MR0">
+<attribute name="NAME" x="349.504" y="-85.725" size="1.778" layer="95" rot="MR0"/>
+<attribute name="VALUE" x="349.504" y="-90.551" size="1.778" layer="96" rot="MR0"/>
+</instance>
+<instance part="VSS33" gate="G$1" x="350.52" y="-93.98" smashed="yes">
+<attribute name="VALUE" x="358.14" y="-93.98" size="1.778" layer="96" rot="R180"/>
 </instance>
 </instances>
@@
 <junction x="360.68" y="-99.06"/>
 <junction x="360.68" y="-76.2"/>
+</segment>
+<segment>
+<wire x1="335.28" y1="-83.82" x2="350.52" y2="-83.82" width="0.1524" layer="91"/>
+<pinref part="C26" gate="G$1" pin="1"/>
+<junction x="335.28" y="-83.82"/>
+<junction x="350.52" y="-83.82"/>
+<label x="337.82" y="-83.82" size="1.778" layer="95"/>
 </segment>
 </net>
@@
 <pinref part="C21" gate="G$1" pin="2"/>
 <pinref part="VSS30" gate="G$1" pin="VSS"/>
+<junction x="350.52" y="-106.68"/>
 </segment>
 <segment>
@@
 <junction x="368.3" y="-76.2"/>
 </segment>
+<segment>
+<pinref part="C26" gate="G$1" pin="2"/>
+<pinref part="VSS33" gate="G$1" pin="VSS"/>
+<junction x="350.52" y="-91.44"/>
+</segment>
 </net>

Commit message: up
Parts:
- removed TP14: PTR1PAD1-13, testpad:PTR1PAD1-13
- added IC2: SFH6916, SFH6916:SFH6916
- added ISO1_R, ISO1_R1: 330 ohm, rcl:R-US_R0805
- added ISO1_R2, ISO1_R3: 2.2k ohm, rcl:R-US_R0805
- added ISO_IO: ISO_IO, con-lstb:MA10-1
- added SW1, SW2: PTS635SL50LFS, PTS635SL50LFS:PTS635SL50LFS
- added U1_TTL: U1_TTL, con-lstb:MA04-1
- renumbered S1 to RESET_SW
Connections:
- new net IOS1_N: IC2.E_4, ISO_IO.1
- new net IOS1_P: IC2.C_4, ISO_IO.2
- new net IOS2_N: IC2.E_3, ISO_IO.3
- new net IOS3_O: IC2.C_2, U1.TDI/RP52/PWM1L/IOMD5/RD3
- new net IOS3_P: ISO1_R3.2, ISO_IO.10
- new net IOS4_O: IC2.C_1, U1.RP53/PCI22/RD4
- new net ISO1_S: ISO1_R.2, U1.TCK/RP50/PWM2L/IOMD3/RD1
- new net ISO2_P: IC2.C_3, ISO_IO.4
- new net ISO2_S: ISO1_R1.2, U1.RP54/ASCL1/RD5
- new net ISO3_N: IC2.K_3, ISO_IO.9
- new net ISO4_N: IC2.K_4, ISO_IO.7
- new net ISO4_P: ISO1_R2.2, ISO_IO.8
- new net N$10: IC2.A_4, ISO1_R2.1
- new net N$7: IC2.A_1, ISO1_R.1
- new net N$8: IC2.A_2, ISO1_R1.1
- new net N$9: IC2.A_3, ISO1_R3.1
- new net SW1: SW1.NO, U1.RP55/ASDA1/RD6
- new net SW2: SW2.NO, U1.RP56/ASCL2/IOMD7/IOMF4/RD7
- new net U1RX: U1.AD2ANN2/AD2AN8/RP24/IOMF0/RB7, U1_TTL.2
- new net U1TX: U1.AD1ANN2/AD1AN8/RP23/RB6, U1_TTL.3
- net VDD: now also U1_TTL.4; no longer TP14.TP
- net VSS: now also IC2.E_1, IC2.E_2, IC2.K_1, IC2.K_2, ISO_IO.5, ISO_IO.6, SW1.COM, SW2.COM, U1_TTL.1
