File: pic32ak_fe.sch (EAGLE design)
At the start: 87 parts, among them IC1 NCP1117LPST33T3G, IC2 SFH6916, J1 CONBNC001, J2 CONBNC001, J3 CONBNC001, J4 CONBNC001, J5 5227222-3, SW1 PTS635SL50LFS, SW2 PTS635SL50LFS, U1 PIC32AK1216GC41064-E/PT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

Commit message: up
Parts:
- added R11, R12, R13: 100 ohm, rcl:R-US_R0805
- added TP14, TP19, TP20, TP21, TP22, TP23, TP24, TP9: PTR1PAD1-13, testpad:PTR1PAD1-13
Connections:
- net IMU_CS: now also TP21.TP
- net SCK2: now also R13.1
- net SCK3: now also TP14.TP
- net SDI2: now also R11.1
- net SDI3: now also TP20.TP
- net SDO2: now also R12.1
- net SDO3: now also TP9.TP
- net VSS: now also R11.2, R12.2, R13.2, TP19.TP, TP22.TP, TP23.TP, TP24.TP
Changed lines of the file:
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@@
 <part name="PWM" library="con-lstb" library_urn="urn:adsk.eagle:library:162" deviceset="MA10-1" device="" package3d_urn="urn:adsk.eagle:package:8346/1" value="PWM"/>
 <part name="VSS38" library="supply1" library_urn="urn:adsk.eagle:library:371" deviceset="VSS" device=""/>
+<part name="TP9" library="testpad" library_urn="urn:adsk.eagle:library:385" deviceset="PTR1" device="PAD1-13" package3d_urn="urn:adsk.eagle:package:27946/1"/>
+<part name="TP14" library="testpad" library_urn="urn:adsk.eagle:library:385" deviceset="PTR1" device="PAD1-13" package3d_urn="urn:adsk.eagle:package:27946/1"/>
+<part name="TP19" library="testpad" library_urn="urn:adsk.eagle:library:385" deviceset="PTR1" device="PAD1-13" package3d_urn="urn:adsk.eagle:package:27946/1"/>
+<part name="TP20" library="testpad" library_urn="urn:adsk.eagle:library:385" deviceset="PTR1" device="PAD1-13" package3d_urn="urn:adsk.eagle:package:27946/1"/>
+<part name="TP21" library="testpad" library_urn="urn:adsk.eagle:library:385" deviceset="PTR1" device="PAD1-13" package3d_urn="urn:adsk.eagle:package:27946/1"/>
+<part name="TP22" library="testpad" library_urn="urn:adsk.eagle:library:385" deviceset="PTR1" device="PAD1-13" package3d_urn="urn:adsk.eagle:package:27946/1"/>
+<part name="TP23" library="testpad" library_urn="urn:adsk.eagle:library:385" deviceset="PTR1" device="PAD1-13" package3d_urn="urn:adsk.eagle:package:27946/1"/>
+<part name="TP24" library="testpad" library_urn="urn:adsk.eagle:library:385" deviceset="PTR1" device="PAD1-13" package3d_urn="urn:adsk.eagle:package:27946/1"/>
+<part name="R11" library="rcl" library_urn="urn:adsk.eagle:library:334" deviceset="R-US_" device="R0805" package3d_urn="urn:adsk.eagle:package:23553/2" value="100 ohm"/>
+<part name="R12" library="rcl" library_urn="urn:adsk.eagle:library:334" deviceset="R-US_" device="R0805" package3d_urn="urn:adsk.eagle:package:23553/2" value="100 ohm"/>
+<part name="R13" library="rcl" library_urn="urn:adsk.eagle:library:334" deviceset="R-US_" device="R0805" package3d_urn="urn:adsk.eagle:package:23553/2" value="100 ohm"/>
+<part name="VSS39" library="supply1" library_urn="urn:adsk.eagle:library:371" deviceset="VSS" device=""/>
 </parts>
 <sheets>
@@
 </instance>
 <instance part="VSS31" gate="G$1" x="246.38" y="-104.14" smashed="yes">
-<attribute name="VALUE" x="254" y="-104.14" size="1.778" layer="96" rot="R180"/>
+<attribute name="VALUE" x="246.38" y="-106.68" size="1.778" layer="96" rot="R180"/>
 </instance>
 <instance part="C23" gate="G$1" x="363.22" y="-99.06" smashed="yes" rot="R90">
@@
 <instance part="VSS38" gate="G$1" x="86.36" y="-127" smashed="yes">
 <attribute name="VALUE" x="83.82" y="-127" size="1.778" layer="96" rot="R180"/>
+</instance>
+<instance part="TP9" gate="G$1" x="332.74" y="-91.44" smashed="yes" rot="R90">
+<attribute name="NAME" x="344.17" y="-89.916" size="1.778" layer="95" rot="R180"/>
+<attribute name="TP_SIGNAL_NAME" x="335.28" y="-90.17" size="1.778" layer="97" rot="R90"/>
+</instance>
+<instance part="TP14" gate="G$1" x="332.74" y="-93.98" smashed="yes" rot="R90">
+<attribute name="NAME" x="344.17" y="-92.456" size="1.778" layer="95" rot="R180"/>
+<attribute name="TP_SIGNAL_NAME" x="335.28" y="-92.71" size="1.778" layer="97" rot="R90"/>
+</instance>
+<instance part="TP19" gate="G$1" x="332.74" y="-104.14" smashed="yes" rot="R90">
+<attribute name="NAME" x="344.17" y="-102.616" size="1.778" layer="95" rot="R180"/>
+<attribute name="TP_SIGNAL_NAME" x="335.28" y="-102.87" size="1.778" layer="97" rot="R90"/>
+</instance>
+<instance part="TP20" gate="G$1" x="261.62" y="-104.14" smashed="yes" rot="R270">
+<attribute name="NAME" x="255.27" y="-108.204" size="1.778" layer="95"/>
+<attribute name="TP_SIGNAL_NAME" x="259.08" y="-105.41" size="1.778" layer="97" rot="R270"/>
+</instance>
+<instance part="TP21" gate="G$1" x="261.62" y="-101.6" smashed="yes" rot="R270">
+<attribute name="NAME" x="250.19" y="-103.124" size="1.778" layer="95"/>
+<attribute name="TP_SIGNAL_NAME" x="259.08" y="-102.87" size="1.778" layer="97" rot="R270"/>
+</instance>
+<instance part="TP22" gate="G$1" x="203.2" y="-48.26" smashed="yes" rot="R180">
+<attribute name="NAME" x="204.216" y="-41.91" size="1.778" layer="95" rot="R270"/>
+<attribute name="TP_SIGNAL_NAME" x="201.93" y="-45.72" size="1.778" layer="97" rot="R180"/>
+</instance>
+<instance part="TP23" gate="G$1" x="198.12" y="-48.26" smashed="yes" rot="R180">
+<attribute name="NAME" x="199.136" y="-41.91" size="1.778" layer="95" rot="R270"/>
+<attribute name="TP_SIGNAL_NAME" x="196.85" y="-45.72" size="1.778" layer="97" rot="R180"/>
+</instance>
+<instance part="TP24" gate="G$1" x="193.04" y="-48.26" smashed="yes" rot="R180">
+<attribute name="NAME" x="194.056" y="-41.91" size="1.778" layer="95" rot="R270"/>
+<attribute name="TP_SIGNAL_NAME" x="191.77" y="-45.72" size="1.778" layer="97" rot="R180"/>
+</instance>
+<instance part="R11" gate="G$1" x="261.62" y="-43.18" smashed="yes" rot="R180">
+<attribute name="NAME" x="265.43" y="-44.6786" size="1.778" layer="95" rot="R180"/>
+<attribute name="VALUE" x="265.43" y="-39.878" size="1.778" layer="96" rot="R180"/>
+</instance>
+<instance part="R12" gate="G$1" x="261.62" y="-48.26" smashed="yes" rot="R180">
+<attribute name="NAME" x="265.43" y="-49.7586" size="1.778" layer="95" rot="R180"/>
+<attribute name="VALUE" x="265.43" y="-44.958" size="1.778" layer="96" rot="R180"/>
+</instance>
+<instance part="R13" gate="G$1" x="261.62" y="-53.34" smashed="yes" rot="R180">
+<attribute name="NAME" x="265.43" y="-54.8386" size="1.778" layer="95" rot="R180"/>
+<attribute name="VALUE" x="265.43" y="-50.038" size="1.778" layer="96" rot="R180"/>
+</instance>
+<instance part="VSS39" gate="G$1" x="256.54" y="-55.88" smashed="yes">
+<attribute name="VALUE" x="254" y="-55.88" size="1.778" layer="96" rot="R180"/>
 </instance>
 </instances>
@@
 <pinref part="VSS28" gate="G$1" pin="VSS"/>
 <junction x="210.82" y="-50.8"/>
+<pinref part="TP22" gate="G$1" pin="TP"/>
+<pinref part="TP23" gate="G$1" pin="TP"/>
+<pinref part="TP24" gate="G$1" pin="TP"/>
+<junction x="193.04" y="-50.8"/>
 </segment>
 <segment>
@@
 <junction x="314.96" y="-104.14"/>
 <junction x="330.2" y="-104.14"/>
-<label x="332.74" y="-104.14" size="1.778" layer="95"/>
+<label x="320.04" y="-104.14" size="1.778" layer="95"/>
+<pinref part="TP19" gate="G$1" pin="TP"/>
 </segment>
 <segment>
@@
 <junction x="86.36" y="-124.46"/>
 </segment>
+<segment>
+<pinref part="R13" gate="G$1" pin="2"/>
+<pinref part="VSS39" gate="G$1" pin="VSS"/>
+<pinref part="R11" gate="G$1" pin="2"/>
+<wire x1="256.54" y1="-53.34" x2="256.54" y2="-48.26" width="0.1524" layer="91"/>
+<junction x="256.54" y="-53.34"/>
+<pinref part="R12" gate="G$1" pin="2"/>
+<wire x1="256.54" y1="-48.26" x2="256.54" y2="-43.18" width="0.1524" layer="91"/>
+<junction x="256.54" y="-48.26"/>
+<junction x="256.54" y="-43.18"/>
+</segment>
 </net>
 <net name="SDI1" class="0">
@@
 <junction x="271.78" y="-66.04"/>
 </segment>
+<segment>
+<wire x1="266.7" y1="-43.18" x2="281.94" y2="-43.18" width="0.1524" layer="91"/>
+<pinref part="R11" gate="G$1" pin="1"/>
+<junction x="266.7" y="-43.18"/>
+<junction x="281.94" y="-43.18"/>
+<label x="269.24" y="-43.18" size="1.778" layer="95"/>
+</segment>
 </net>
 <net name="SDO2" class="0">
@@
 <pinref part="TP1" gate="G$1" pin="TP"/>
 </segment>
+<segment>
+<wire x1="281.94" y1="-48.26" x2="266.7" y2="-48.26" width="0.1524" layer="91"/>
+<pinref part="R12" gate="G$1" pin="1"/>
+<junction x="266.7" y="-48.26"/>
+<junction x="281.94" y="-48.26"/>
+<label x="269.24" y="-48.26" size="1.778" layer="95"/>
+</segment>
 </net>
 <net name="SCK2" class="0">
@@
 <label x="325.12" y="-68.58" size="1.778" layer="95"/>
 <pinref part="TP2" gate="G$1" pin="TP"/>
+</segment>
+<segment>
+<wire x1="266.7" y1="-53.34" x2="281.94" y2="-53.34" width="0.1524" layer="91"/>
+<pinref part="R13" gate="G$1" pin="1"/>
+<junction x="266.7" y="-53.34"/>
+<junction x="281.94" y="-53.34"/>
+<label x="269.24" y="-53.34" size="1.778" layer="95"/>
 </segment>
 </net>
@@
 <junction x="279.4" y="-101.6"/>
 <junction x="264.16" y="-101.6"/>
-<label x="254" y="-101.6" size="1.778" layer="95"/>
+<label x="269.24" y="-101.6" size="1.778" layer="95"/>
+<pinref part="TP21" gate="G$1" pin="TP"/>
 </segment>
 </net>
@@
 <junction x="279.4" y="-104.14"/>
 <junction x="264.16" y="-104.14"/>
-<label x="256.54" y="-104.14" size="1.778" layer="95"/>
+<label x="271.78" y="-104.14" size="1.778" layer="95"/>
+<pinref part="TP20" gate="G$1" pin="TP"/>
 </segment>
 </net>
@@
 <junction x="314.96" y="-91.44"/>
 <junction x="330.2" y="-91.44"/>
-<label x="332.74" y="-91.44" size="1.778" layer="95"/>
+<label x="320.04" y="-91.44" size="1.778" layer="95"/>
+<pinref part="TP9" gate="G$1" pin="TP"/>
 </segment>
 </net>
@@
 <junction x="314.96" y="-93.98"/>
 <junction x="330.2" y="-93.98"/>
-<label x="332.74" y="-93.98" size="1.778" layer="95"/>
-</segment>
-</net>
+<label x="320.04" y="-93.98" size="1.778" layer="95"/>
+<pinref part="TP14" gate="G$1" pin="TP"/>
+</segment>
+</net>

Commit message: up
Parts:
- added AVDD_JUMPER: AVDD JUMPER, jumper:SJ2W
- added C27, C28: 0.1uf, rcl:C-USC0603
- added IC3: NCP51460SN33T1G, NCP51460SN33T1G:NCP51460SN33T1G
Connections:
- new net 3.3REG: AVDD_JUMPER.1, IC3.VOUT
- new net AVDD_IN: AVDD_JUMPER.2, C28.1, E1.1
- net VDD: now also AVDD_JUMPER.3; no longer E1.1
- net VIN: now also C27.1, IC3.VIN
- net VSS: now also C27.2, C28.2, IC3.GND
Changed lines of the file:
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@@
 <part name="R13" library="rcl" library_urn="urn:adsk.eagle:library:334" deviceset="R-US_" device="R0805" package3d_urn="urn:adsk.eagle:package:23553/2" value="100 ohm"/>
 <part name="VSS39" library="supply1" library_urn="urn:adsk.eagle:library:371" deviceset="VSS" device=""/>
+<part name="IC3" library="NCP51460SN33T1G" deviceset="NCP51460SN33T1G" device=""/>
+<part name="VSS40" library="supply1" library_urn="urn:adsk.eagle:library:371" deviceset="VSS" device=""/>
+<part name="AVDD_JUMPER" library="jumper" library_urn="urn:adsk.eagle:library:252" deviceset="SJ2W" device="" package3d_urn="urn:adsk.eagle:package:15474/1" value="AVDD JUMPER"/>
+<part name="C27" library="rcl" library_urn="urn:adsk.eagle:library:334" deviceset="C-US" device="C0603" package3d_urn="urn:adsk.eagle:package:23616/2" value="0.1uf"/>
+<part name="VSS41" library="supply1" library_urn="urn:adsk.eagle:library:371" deviceset="VSS" device=""/>
+<part name="C28" library="rcl" library_urn="urn:adsk.eagle:library:334" deviceset="C-US" device="C0603" package3d_urn="urn:adsk.eagle:package:23616/2" value="0.1uf"/>
+<part name="VSS42" library="supply1" library_urn="urn:adsk.eagle:library:371" deviceset="VSS" device=""/>
 </parts>
 <sheets>
@@
 </instance>
 <instance part="ISO1_R" gate="G$1" x="139.7" y="-96.52" smashed="yes" rot="R180">
-<attribute name="NAME" x="143.51" y="-90.3986" size="1.778" layer="95" rot="R180"/>
-<attribute name="VALUE" x="143.51" y="-93.218" size="1.778" layer="96" rot="R180"/>
+<attribute name="NAME" x="115.57" y="-95.4786" size="1.778" layer="95" rot="R180"/>
+<attribute name="VALUE" x="143.51" y="-98.298" size="1.778" layer="96" rot="R180"/>
 </instance>
 <instance part="ISO1_R1" gate="G$1" x="139.7" y="-101.6" smashed="yes" rot="R180">
-<attribute name="NAME" x="143.51" y="-95.4786" size="1.778" layer="95" rot="R180"/>
-<attribute name="VALUE" x="143.51" y="-98.298" size="1.778" layer="96" rot="R180"/>
+<attribute name="NAME" x="115.57" y="-100.5586" size="1.778" layer="95" rot="R180"/>
+<attribute name="VALUE" x="143.51" y="-103.378" size="1.778" layer="96" rot="R180"/>
 </instance>
 <instance part="ISO1_R3" gate="G$1" x="139.7" y="-106.68" smashed="yes" rot="R180">
-<attribute name="NAME" x="143.51" y="-100.5586" size="1.778" layer="95" rot="R180"/>
-<attribute name="VALUE" x="143.51" y="-103.378" size="1.778" layer="96" rot="R180"/>
+<attribute name="NAME" x="115.57" y="-105.6386" size="1.778" layer="95" rot="R180"/>
+<attribute name="VALUE" x="143.51" y="-108.458" size="1.778" layer="96" rot="R180"/>
 </instance>
 <instance part="ISO1_R2" gate="G$1" x="139.7" y="-111.76" smashed="yes" rot="R180">
-<attribute name="NAME" x="143.51" y="-105.6386" size="1.778" layer="95" rot="R180"/>
-<attribute name="VALUE" x="143.51" y="-108.458" size="1.778" layer="96" rot="R180"/>
+<attribute name="NAME" x="115.57" y="-110.7186" size="1.778" layer="95" rot="R180"/>
+<attribute name="VALUE" x="143.51" y="-113.538" size="1.778" layer="96" rot="R180"/>
 </instance>
 <instance part="U1_TTL" gate="1" x="45.72" y="-50.8" smashed="yes">
@@
 <instance part="VSS39" gate="G$1" x="256.54" y="-55.88" smashed="yes">
 <attribute name="VALUE" x="254" y="-55.88" size="1.778" layer="96" rot="R180"/>
+</instance>
+<instance part="IC3" gate="G$1" x="7.62" y="111.76" smashed="yes">
+<attribute name="NAME" x="31.75" y="119.38" size="1.778" layer="95" align="center-left"/>
+<attribute name="VALUE" x="31.75" y="116.84" size="1.778" layer="96" align="center-left"/>
+</instance>
+<instance part="VSS40" gate="G$1" x="35.56" y="109.22" smashed="yes">
+<attribute name="VALUE" x="33.02" y="109.22" size="1.778" layer="96" rot="R180"/>
+</instance>
+<instance part="AVDD_JUMPER" gate="G$1" x="50.8" y="109.22" smashed="yes" rot="R180">
+<attribute name="NAME" x="71.12" y="106.299" size="1.778" layer="95" rot="R180"/>
+<attribute name="VALUE" x="71.12" y="113.665" size="1.778" layer="96" rot="R180"/>
+</instance>
+<instance part="C27" gate="G$1" x="-7.62" y="109.22" smashed="yes" rot="MR0">
+<attribute name="NAME" x="-8.636" y="109.855" size="1.778" layer="95" rot="MR0"/>
+<attribute name="VALUE" x="-8.636" y="105.029" size="1.778" layer="96" rot="MR0"/>
+</instance>
+<instance part="VSS41" gate="G$1" x="-7.62" y="101.6" smashed="yes">
+<attribute name="VALUE" x="-10.16" y="101.6" size="1.778" layer="96" rot="R180"/>
+</instance>
+<instance part="C28" gate="G$1" x="63.5" y="106.68" smashed="yes" rot="MR0">
+<attribute name="NAME" x="62.484" y="107.315" size="1.778" layer="95" rot="MR0"/>
+<attribute name="VALUE" x="62.484" y="102.489" size="1.778" layer="96" rot="MR0"/>
+</instance>
+<instance part="VSS42" gate="G$1" x="63.5" y="99.06" smashed="yes">
+<attribute name="VALUE" x="60.96" y="99.06" size="1.778" layer="96" rot="R180"/>
 </instance>
 </instances>
@@
 <junction x="317.5" y="83.82"/>
 <junction x="317.5" y="96.52"/>
-</segment>
-<segment>
-<wire x1="63.5" y1="109.22" x2="78.74" y2="109.22" width="0.1524" layer="91"/>
-<pinref part="E1" gate="G$1" pin="1"/>
-<junction x="78.74" y="109.22"/>
-<junction x="63.5" y="109.22"/>
-<label x="66.04" y="109.22" size="1.778" layer="95"/>
 </segment>
 <segment>
@@
 <junction x="350.52" y="-83.82"/>
 <label x="337.82" y="-83.82" size="1.778" layer="95"/>
+</segment>
+<segment>
+<wire x1="50.8" y1="114.3" x2="66.04" y2="114.3" width="0.1524" layer="91"/>
+<pinref part="AVDD_JUMPER" gate="G$1" pin="3"/>
+<junction x="66.04" y="114.3"/>
+<junction x="50.8" y="114.3"/>
+<label x="58.42" y="114.3" size="1.778" layer="95"/>
 </segment>
 </net>
@@
 <junction x="256.54" y="-43.18"/>
 </segment>
+<segment>
+<pinref part="IC3" gate="G$1" pin="GND"/>
+<pinref part="VSS40" gate="G$1" pin="VSS"/>
+<junction x="35.56" y="111.76"/>
+</segment>
+<segment>
+<pinref part="C27" gate="G$1" pin="2"/>
+<pinref part="VSS41" gate="G$1" pin="VSS"/>
+<junction x="-7.62" y="104.14"/>
+</segment>
+<segment>
+<pinref part="C28" gate="G$1" pin="2"/>
+<pinref part="VSS42" gate="G$1" pin="VSS"/>
+<junction x="63.5" y="101.6"/>
+</segment>
 </net>
 <net name="SDI1" class="0">
@@
 <junction x="363.22" y="86.36"/>
 <label x="365.76" y="86.36" size="1.778" layer="95"/>
+</segment>
+<segment>
+<wire x1="7.62" y1="111.76" x2="-7.62" y2="111.76" width="0.1524" layer="91"/>
+<pinref part="IC3" gate="G$1" pin="VIN"/>
+<junction x="7.62" y="111.76"/>
+<junction x="-7.62" y="111.76"/>
+<label x="-2.54" y="111.76" size="1.778" layer="95"/>
+<pinref part="C27" gate="G$1" pin="1"/>
 </segment>
 </net>
@@
 </segment>
 </net>
+<net name="3.3REG" class="1">
+<segment>
+<pinref part="IC3" gate="G$1" pin="VOUT"/>
+<wire x1="7.62" y1="109.22" x2="2.54" y2="109.22" width="0.1524" layer="91"/>
+<junction x="7.62" y="109.22"/>
+<junction x="2.54" y="109.22"/>
+<label x="-2.54" y="106.68" size="1.778" layer="95"/>
+</segment>
+<segment>
+<wire x1="50.8" y1="104.14" x2="45.72" y2="104.14" width="0.1524" layer="91"/>
+<pinref part="AVDD_JUMPER" gate="G$1" pin="1"/>
+<junction x="45.72" y="104.14"/>
+<junction x="50.8" y="104.14"/>
+<label x="35.56" y="104.14" size="1.778" layer="95"/>
+</segment>
+</net>
+<net name="AVDD_IN" class="1">
+<segment>
+<pinref part="E1" gate="G$1" pin="1"/>
+<pinref part="AVDD_JUMPER" gate="G$1" pin="2"/>
+<wire x1="78.74" y1="109.22" x2="63.5" y2="109.22" width="0.1524" layer="91"/>
+<junction x="55.88" y="109.22"/>
+<junction x="78.74" y="109.22"/>
+<label x="63.5" y="109.22" size="1.778" layer="95"/>
+<pinref part="C28" gate="G$1" pin="1"/>
+<wire x1="63.5" y1="109.22" x2="55.88" y2="109.22" width="0.1524" layer="91"/>
+<junction x="63.5" y="109.22"/>
+</segment>
+</net>
