File: pic32ak_fe.sch (EAGLE design)
At the start: 103 parts, among them IC1 NCP1117LPST33T3G, IC2 SFH6916, IC3 NCP51460SN33T1G, J1 CONBNC001, J2 CONBNC001, J3 CONBNC001, J4 CONBNC001, J5 5227222-3, SW1 PTS635SL50LFS, SW2 PTS635SL50LFS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

Commit message: finish V1.1 board
Parts:
- added C29: 0.1uf, rcl:C-USC0603
- R11, R12, R13: device rcl:R-US_R0805 -> rcl:R-US_R0603
Connections:
- net RESET_SW: now also C29.1
- net SCK2: now also R13.2; no longer R13.1
- net SDI2: now also R11.2; no longer R11.1
- net SDO2: now also R12.2; no longer R12.1
- net VSS: now also C29.2, R11.1, R12.1, R13.1; no longer R11.2, R12.2, R13.2
Other:
- moved on the sheet: R11, R12, R13
Changed lines of the file:
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@@
 <part name="TP23" library="testpad" library_urn="urn:adsk.eagle:library:385" deviceset="PTR1" device="PAD1-13" package3d_urn="urn:adsk.eagle:package:27946/1"/>
 <part name="TP24" library="testpad" library_urn="urn:adsk.eagle:library:385" deviceset="PTR1" device="PAD1-13" package3d_urn="urn:adsk.eagle:package:27946/1"/>
-<part name="R11" library="rcl" library_urn="urn:adsk.eagle:library:334" deviceset="R-US_" device="R0805" package3d_urn="urn:adsk.eagle:package:23553/2" value="50 ohm"/>
-<part name="R12" library="rcl" library_urn="urn:adsk.eagle:library:334" deviceset="R-US_" device="R0805" package3d_urn="urn:adsk.eagle:package:23553/2" value="50 ohm"/>
-<part name="R13" library="rcl" library_urn="urn:adsk.eagle:library:334" deviceset="R-US_" device="R0805" package3d_urn="urn:adsk.eagle:package:23553/2" value="50 ohm"/>
 <part name="VSS39" library="supply1" library_urn="urn:adsk.eagle:library:371" deviceset="VSS" device=""/>
 <part name="IC3" library="NCP51460SN33T1G" deviceset="NCP51460SN33T1G" device=""/>
@@
 <part name="USBC-PWR" library="con-lstb" library_urn="urn:adsk.eagle:library:162" deviceset="MA04-1" device="" package3d_urn="urn:adsk.eagle:package:8337/1" value="USBC-PWR"/>
 <part name="VSS43" library="supply1" library_urn="urn:adsk.eagle:library:371" deviceset="VSS" device=""/>
+<part name="R11" library="rcl" library_urn="urn:adsk.eagle:library:334" deviceset="R-US_" device="R0603" package3d_urn="urn:adsk.eagle:package:23555/3" value="50 ohm"/>
+<part name="R12" library="rcl" library_urn="urn:adsk.eagle:library:334" deviceset="R-US_" device="R0603" package3d_urn="urn:adsk.eagle:package:23555/3" value="50 ohm"/>
+<part name="R13" library="rcl" library_urn="urn:adsk.eagle:library:334" deviceset="R-US_" device="R0603" package3d_urn="urn:adsk.eagle:package:23555/3" value="50 ohm"/>
+<part name="C29" library="rcl" library_urn="urn:adsk.eagle:library:334" deviceset="C-US" device="C0603" package3d_urn="urn:adsk.eagle:package:23616/2" value="0.1uf"/>
+<part name="VSS44" library="supply1" library_urn="urn:adsk.eagle:library:371" deviceset="VSS" device=""/>
 </parts>
 <sheets>
@@
 <attribute name="TP_SIGNAL_NAME" x="191.77" y="-45.72" size="1.778" layer="97" rot="R180"/>
 </instance>
-<instance part="R11" gate="G$1" x="261.62" y="-43.18" smashed="yes" rot="R180">
-<attribute name="NAME" x="262.89" y="-39.5986" size="1.778" layer="95" rot="R180"/>
-<attribute name="VALUE" x="255.27" y="-39.878" size="1.778" layer="96" rot="R180"/>
-</instance>
-<instance part="R12" gate="G$1" x="261.62" y="-48.26" smashed="yes" rot="R180">
-<attribute name="NAME" x="262.89" y="-44.6786" size="1.778" layer="95" rot="R180"/>
-<attribute name="VALUE" x="255.27" y="-44.958" size="1.778" layer="96" rot="R180"/>
-</instance>
-<instance part="R13" gate="G$1" x="261.62" y="-53.34" smashed="yes" rot="R180">
-<attribute name="NAME" x="262.89" y="-49.7586" size="1.778" layer="95" rot="R180"/>
-<attribute name="VALUE" x="255.27" y="-50.038" size="1.778" layer="96" rot="R180"/>
-</instance>
 <instance part="VSS39" gate="G$1" x="256.54" y="-55.88" smashed="yes">
 <attribute name="VALUE" x="254" y="-55.88" size="1.778" layer="96" rot="R180"/>
@@
 <instance part="VSS43" gate="G$1" x="43.18" y="-106.68" smashed="yes">
 <attribute name="VALUE" x="40.64" y="-106.68" size="1.778" layer="96" rot="R180"/>
+</instance>
+<instance part="R11" gate="G$1" x="261.62" y="-43.18" smashed="yes">
+<attribute name="NAME" x="257.81" y="-41.6814" size="1.778" layer="95"/>
+<attribute name="VALUE" x="245.11" y="-43.942" size="1.778" layer="96"/>
+</instance>
+<instance part="R12" gate="G$1" x="261.62" y="-48.26" smashed="yes">
+<attribute name="NAME" x="257.81" y="-46.7614" size="1.778" layer="95"/>
+<attribute name="VALUE" x="245.11" y="-49.022" size="1.778" layer="96"/>
+</instance>
+<instance part="R13" gate="G$1" x="261.62" y="-53.34" smashed="yes">
+<attribute name="NAME" x="257.81" y="-51.8414" size="1.778" layer="95"/>
+<attribute name="VALUE" x="245.11" y="-54.102" size="1.778" layer="96"/>
+</instance>
+<instance part="C29" gate="G$1" x="314.96" y="55.88" smashed="yes" rot="MR0">
+<attribute name="NAME" x="321.564" y="56.515" size="1.778" layer="95" rot="MR0"/>
+<attribute name="VALUE" x="324.104" y="54.229" size="1.778" layer="96" rot="MR0"/>
+</instance>
+<instance part="VSS44" gate="G$1" x="314.96" y="48.26" smashed="yes">
+<attribute name="VALUE" x="312.42" y="48.26" size="1.778" layer="96" rot="R180"/>
 </instance>
 </instances>
@@
 </segment>
 <segment>
-<pinref part="R13" gate="G$1" pin="2"/>
 <pinref part="VSS39" gate="G$1" pin="VSS"/>
-<pinref part="R11" gate="G$1" pin="2"/>
 <wire x1="256.54" y1="-53.34" x2="256.54" y2="-48.26" width="0.1524" layer="91"/>
-<junction x="256.54" y="-53.34"/>
-<pinref part="R12" gate="G$1" pin="2"/>
+<pinref part="R11" gate="G$1" pin="1"/>
+<pinref part="R12" gate="G$1" pin="1"/>
 <wire x1="256.54" y1="-48.26" x2="256.54" y2="-43.18" width="0.1524" layer="91"/>
 <junction x="256.54" y="-48.26"/>
+<pinref part="R13" gate="G$1" pin="1"/>
+<junction x="256.54" y="-53.34"/>
 <junction x="256.54" y="-43.18"/>
 </segment>
@@
 <pinref part="VSS43" gate="G$1" pin="VSS"/>
 <junction x="43.18" y="-104.14"/>
+</segment>
+<segment>
+<pinref part="C29" gate="G$1" pin="2"/>
+<pinref part="VSS44" gate="G$1" pin="VSS"/>
+<junction x="314.96" y="50.8"/>
 </segment>
 </net>
@@
 <segment>
 <wire x1="266.7" y1="-43.18" x2="281.94" y2="-43.18" width="0.1524" layer="91"/>
-<pinref part="R11" gate="G$1" pin="1"/>
-<junction x="266.7" y="-43.18"/>
 <junction x="281.94" y="-43.18"/>
 <label x="269.24" y="-43.18" size="1.778" layer="95"/>
+<pinref part="R11" gate="G$1" pin="2"/>
+<junction x="266.7" y="-43.18"/>
 </segment>
 </net>
@@
 <segment>
 <wire x1="281.94" y1="-48.26" x2="266.7" y2="-48.26" width="0.1524" layer="91"/>
-<pinref part="R12" gate="G$1" pin="1"/>
-<junction x="266.7" y="-48.26"/>
 <junction x="281.94" y="-48.26"/>
 <label x="269.24" y="-48.26" size="1.778" layer="95"/>
+<pinref part="R12" gate="G$1" pin="2"/>
+<junction x="266.7" y="-48.26"/>
 </segment>
 </net>
@@
 <segment>
 <wire x1="266.7" y1="-53.34" x2="281.94" y2="-53.34" width="0.1524" layer="91"/>
-<pinref part="R13" gate="G$1" pin="1"/>
-<junction x="266.7" y="-53.34"/>
 <junction x="281.94" y="-53.34"/>
 <label x="269.24" y="-53.34" size="1.778" layer="95"/>
+<pinref part="R13" gate="G$1" pin="2"/>
+<junction x="266.7" y="-53.34"/>
 </segment>
 </net>
@@
 <pinref part="C16" gate="G$1" pin="1"/>
 <junction x="307.34" y="58.42"/>
-<wire x1="307.34" y1="58.42" x2="325.12" y2="58.42" width="0.1524" layer="91"/>
+<wire x1="307.34" y1="58.42" x2="314.96" y2="58.42" width="0.1524" layer="91"/>
 <junction x="325.12" y="58.42"/>
 <label x="314.96" y="60.96" size="1.778" layer="95"/>
-</segment>
-<segment>
+<pinref part="C29" gate="G$1" pin="1"/>
+<wire x1="314.96" y1="58.42" x2="325.12" y2="58.42" width="0.1524" layer="91"/>
+<junction x="314.96" y="58.42"/>
+</segment>
+<segment>

Commit message: up
Parts:
- added TEST_P1: PTR1PAD1-20, testpad:PTR1PAD1-20
Connections:
- net TEST_P1: now also TEST_P1.TP
Changed lines of the file:
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@@
 <part name="C29" library="rcl" library_urn="urn:adsk.eagle:library:334" deviceset="C-US" device="C0603" package3d_urn="urn:adsk.eagle:package:23616/2" value="0.1uf"/>
 <part name="VSS44" library="supply1" library_urn="urn:adsk.eagle:library:371" deviceset="VSS" device=""/>
+<part name="TEST_P1" library="testpad" library_urn="urn:adsk.eagle:library:385" deviceset="PTR1" device="PAD1-20" package3d_urn="urn:adsk.eagle:package:27950/1"/>
 </parts>
 <sheets>
@@
 </instance>
 <instance part="VSS38" gate="G$1" x="86.36" y="-127" smashed="yes">
-<attribute name="VALUE" x="83.82" y="-127" size="1.778" layer="96" rot="R180"/>
+<attribute name="VALUE" x="93.98" y="-124.46" size="1.778" layer="96" rot="R180"/>
 </instance>
 <instance part="TP9" gate="G$1" x="332.74" y="-91.44" smashed="yes" rot="R90">
@@
 <instance part="VSS44" gate="G$1" x="314.96" y="48.26" smashed="yes">
 <attribute name="VALUE" x="312.42" y="48.26" size="1.778" layer="96" rot="R180"/>
+</instance>
+<instance part="TEST_P1" gate="G$1" x="99.06" y="-99.06" smashed="yes" rot="R180">
+<attribute name="NAME" x="87.63" y="-98.044" size="1.778" layer="95"/>
+<attribute name="TP_SIGNAL_NAME" x="97.79" y="-96.52" size="1.778" layer="97" rot="R180"/>
 </instance>
 </instances>
@@
 </segment>
 <segment>
-<wire x1="101.6" y1="-101.6" x2="86.36" y2="-101.6" width="0.1524" layer="91"/>
+<wire x1="101.6" y1="-101.6" x2="99.06" y2="-101.6" width="0.1524" layer="91"/>
 <pinref part="PWM" gate="1" pin="10"/>
 <junction x="86.36" y="-101.6"/>
 <junction x="101.6" y="-101.6"/>
 <label x="91.44" y="-101.6" size="1.778" layer="95"/>
-</segment>
-</net>
+<pinref part="TEST_P1" gate="G$1" pin="TP"/>
+<wire x1="99.06" y1="-101.6" x2="86.36" y2="-101.6" width="0.1524" layer="91"/>
+<junction x="99.06" y="-101.6"/>
+</segment>
+</net>

Commit message: up
Connections:
- net RB1_DU renamed RB1
Changed lines of the file:
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@@
 <pinref part="C13" gate="G$1" pin="2"/>
 <pinref part="VSS4" gate="G$1" pin="VSS"/>
+<junction x="149.86" y="81.28"/>
 </segment>
 <segment>
@@
 <pinref part="C17" gate="G$1" pin="2"/>
 <pinref part="VSS13" gate="G$1" pin="VSS"/>
+<junction x="43.18" y="-81.28"/>
 </segment>
 <segment>
 <pinref part="C18" gate="G$1" pin="2"/>
 <pinref part="VSS14" gate="G$1" pin="VSS"/>
+<junction x="30.48" y="-78.74"/>
 </segment>
 <segment>
@@
 <pinref part="C22" gate="G$1" pin="2"/>
 <pinref part="VSS31" gate="G$1" pin="VSS"/>
+<junction x="246.38" y="-101.6"/>
 </segment>
 <segment>
@@
 <junction x="86.36" y="81.28"/>
 <junction x="86.36" y="73.66"/>
-<label x="83.82" y="68.58" size="1.778" layer="95"/>
+<label x="83.82" y="71.12" size="1.778" layer="95"/>
 <pinref part="C9" gate="G$1" pin="2"/>
 <wire x1="86.36" y1="81.28" x2="86.36" y2="93.98" width="0.1524" layer="91"/>
@@
 </segment>
 </net>
-<net name="RB1_DU" class="0">
+<net name="RB1" class="0">
 <segment>
 <pinref part="U1" gate="A" pin="TMS/OA2IN-/AD1AN4/AD2ANN1/RP18/RB1"/>
