File: pic32ak_fe.sch (EAGLE design)
At the start: 105 parts, among them IC1 NCP1117LPST33T3G, IC2 SFH6916, IC3 NCP51460SN33T1G, J1 CONBNC001, J2 CONBNC001, J3 CONBNC001, J4 CONBNC001, J5 5227222-3, SW1 PTS635SL50LFS, SW2 PTS635SL50LFS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

Commit message: up
Connections:
- net RC8 renamed RC6
Changed lines of the file:
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@@
 </segment>
 </net>
-<net name="RC8" class="0">
+<net name="RC6" class="0">
 <segment>
 <pinref part="U1" gate="A" pin="RP39/RC6"/>

Commit message: up PCB
Parts:
- added EXT_SW: EXT_SW, pinhead:PINHD-2X2
Connections:
- net SW1: now also EXT_SW.1
- net SW2: now also EXT_SW.2
- net VSS: now also EXT_SW.3, EXT_SW.4
Changed lines of the file:
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@@
 <part name="VSS44" library="supply1" library_urn="urn:adsk.eagle:library:371" deviceset="VSS" device=""/>
 <part name="TEST_P1" library="testpad" library_urn="urn:adsk.eagle:library:385" deviceset="PTR1" device="PAD1-20" package3d_urn="urn:adsk.eagle:package:27950/1"/>
+<part name="EXT_SW" library="pinhead" library_urn="urn:adsk.eagle:library:325" deviceset="PINHD-2X2" device="" package3d_urn="urn:adsk.eagle:package:22455/2" value="EXT_SW"/>
+<part name="VSS45" library="supply1" library_urn="urn:adsk.eagle:library:371" deviceset="VSS" device=""/>
+<part name="VSS46" library="supply1" library_urn="urn:adsk.eagle:library:371" deviceset="VSS" device=""/>
 </parts>
 <sheets>
@@
 <attribute name="NAME" x="87.63" y="-98.044" size="1.778" layer="95"/>
 <attribute name="TP_SIGNAL_NAME" x="97.79" y="-96.52" size="1.778" layer="97" rot="R180"/>
+</instance>
+<instance part="EXT_SW" gate="A" x="355.6" y="0" smashed="yes">
+<attribute name="NAME" x="346.71" y="5.715" size="1.778" layer="95"/>
+<attribute name="VALUE" x="349.25" y="-10.16" size="1.778" layer="96"/>
+</instance>
+<instance part="VSS45" gate="G$1" x="350.52" y="-2.54" smashed="yes">
+<attribute name="VALUE" x="353.06" y="-5.08" size="1.778" layer="96" rot="R180"/>
+</instance>
+<instance part="VSS46" gate="G$1" x="358.14" y="-2.54" smashed="yes">
+<attribute name="VALUE" x="360.68" y="-5.08" size="1.778" layer="96" rot="R180"/>
 </instance>
 </instances>
@@
 <junction x="314.96" y="50.8"/>
 </segment>
+<segment>
+<pinref part="EXT_SW" gate="A" pin="3"/>
+<pinref part="VSS45" gate="G$1" pin="VSS"/>
+<junction x="350.52" y="0"/>
+</segment>
+<segment>
+<pinref part="EXT_SW" gate="A" pin="4"/>
+<pinref part="VSS46" gate="G$1" pin="VSS"/>
+<junction x="358.14" y="0"/>
+</segment>
 </net>
 <net name="SDI1" class="0">
@@
 <label x="365.76" y="38.1" size="1.778" layer="95"/>
 </segment>
+<segment>
+<wire x1="342.9" y1="2.54" x2="350.52" y2="2.54" width="0.1524" layer="91"/>
+<pinref part="EXT_SW" gate="A" pin="1"/>
+<junction x="342.9" y="2.54"/>
+<junction x="350.52" y="2.54"/>
+<label x="335.28" y="2.54" size="1.778" layer="95"/>
+</segment>
 </net>
 <net name="SW2" class="0">
@@
 <label x="365.76" y="22.86" size="1.778" layer="95"/>
 </segment>
-</net>
+<segment>
+<wire x1="358.14" y1="2.54" x2="365.76" y2="2.54" width="0.1524" layer="91"/>
+<pinref part="EXT_SW" gate="A" pin="2"/>
+<junction x="358.14" y="2.54"/>
+<junction x="365.76" y="2.54"/>
+<label x="368.3" y="2.54" size="1.778" layer="95"/>
+</segment>
+</net>

Commit message: up
Parts:
- added BISS-C: BISS-C, con-lstb:MA10-1
- added BISS_DE1: BISS_DE1, jumper:SJ2W
- added BISS_DE2: BISS_DE2, jumper:SJ2W
- added C30: 0.1uf, rcl:C-USC0603
- added C31: 1000pf, rcl:C-USC0603
- added IC4: SN65C1168EPWR, SN65C1168EPWR:SN65C1168EPWR
- added RS422_IN: PTR1PAD1-13, testpad:PTR1PAD1-13
Connections:
- new net MA+: BISS-C.6, IC4.1Z
- new net MA-: BISS-C.7, IC4.1Y
- new net MO+: BISS-C.4, IC4.2Z
- new net MO-: BISS-C.5, IC4.2Y
- new net N$11: BISS_DE1.2, IC4.!RE
- new net N$12: BISS_DE2.2, IC4.DE
- new net N$19: IC4.2R, RS422_IN.TP
- new net RS422_I+: BISS-C.2, IC4.2B
- new net RS422_I-: BISS-C.3, IC4.2A
- new net SL+: BISS-C.8, IC4.1B
- new net SL-: BISS-C.9, IC4.1A
- net RA6: now also IC4.2D
- net RB1: now also IC4.ID
- net RD2: now also IC4.1R
- net VIN: now also BISS-C.10, BISS_DE1.3, BISS_DE2.1, C30.1, C31.1, IC4.VCC
- net VSS: now also BISS-C.1, BISS_DE1.1, BISS_DE2.3, C30.2, C31.2, IC4.GND

Commit message: up
Parts:
- added C32: 10uf, rcl:C-USC0805
- added R14, R15, R16, R17: 120 ohm, rcl:R-US_R0603
Connections:
- net MA+: now also R15.2
- net MA-: now also R15.1
- net MO+: now also R16.2
- net MO-: now also R16.1
- net RS422_I+: now also R17.2
- net RS422_I-: now also R17.1
- net SL+: now also R14.2
- net SL-: now also R14.1
- net VIN: now also C32.1
- net VSS: now also C32.2
Changed lines of the file:
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@@
 <part name="VSS52" library="supply1" library_urn="urn:adsk.eagle:library:371" deviceset="VSS" device=""/>
 <part name="RS422_IN" library="testpad" library_urn="urn:adsk.eagle:library:385" deviceset="PTR1" device="PAD1-13" package3d_urn="urn:adsk.eagle:package:27946/1"/>
+<part name="R14" library="rcl" library_urn="urn:adsk.eagle:library:334" deviceset="R-US_" device="R0603" package3d_urn="urn:adsk.eagle:package:23555/3" value="120 ohm"/>
+<part name="R15" library="rcl" library_urn="urn:adsk.eagle:library:334" deviceset="R-US_" device="R0603" package3d_urn="urn:adsk.eagle:package:23555/3" value="120 ohm"/>
+<part name="R16" library="rcl" library_urn="urn:adsk.eagle:library:334" deviceset="R-US_" device="R0603" package3d_urn="urn:adsk.eagle:package:23555/3" value="120 ohm"/>
+<part name="R17" library="rcl" library_urn="urn:adsk.eagle:library:334" deviceset="R-US_" device="R0603" package3d_urn="urn:adsk.eagle:package:23555/3" value="120 ohm"/>
+<part name="C32" library="rcl" library_urn="urn:adsk.eagle:library:334" deviceset="C-US" device="C0805" package3d_urn="urn:adsk.eagle:package:23617/2" value="10uf"/>
+<part name="VSS53" library="supply1" library_urn="urn:adsk.eagle:library:371" deviceset="VSS" device=""/>
 </parts>
 <sheets>
@@
 <attribute name="NAME" x="140.97" y="112.776" size="1.778" layer="95"/>
 <attribute name="TP_SIGNAL_NAME" x="144.78" y="110.49" size="1.778" layer="97" rot="R270"/>
+</instance>
+<instance part="R14" gate="G$1" x="144.78" y="58.42" smashed="yes">
+<attribute name="NAME" x="140.97" y="59.9186" size="1.778" layer="95"/>
+<attribute name="VALUE" x="138.43" y="55.118" size="1.778" layer="96"/>
+</instance>
+<instance part="R15" gate="G$1" x="160.02" y="58.42" smashed="yes">
+<attribute name="NAME" x="156.21" y="59.9186" size="1.778" layer="95"/>
+<attribute name="VALUE" x="153.67" y="55.118" size="1.778" layer="96"/>
+</instance>
+<instance part="R16" gate="G$1" x="175.26" y="58.42" smashed="yes">
+<attribute name="NAME" x="171.45" y="59.9186" size="1.778" layer="95"/>
+<attribute name="VALUE" x="168.91" y="55.118" size="1.778" layer="96"/>
+</instance>
+<instance part="R17" gate="G$1" x="127" y="58.42" smashed="yes">
+<attribute name="NAME" x="123.19" y="59.9186" size="1.778" layer="95"/>
+<attribute name="VALUE" x="120.65" y="55.118" size="1.778" layer="96"/>
+</instance>
+<instance part="C32" gate="G$1" x="223.52" y="119.38" smashed="yes">
+<attribute name="NAME" x="224.536" y="120.015" size="1.778" layer="95"/>
+<attribute name="VALUE" x="224.536" y="115.189" size="1.778" layer="96"/>
+</instance>
+<instance part="VSS53" gate="G$1" x="223.52" y="111.76" smashed="yes">
+<attribute name="VALUE" x="220.98" y="111.76" size="1.778" layer="96" rot="R180"/>
 </instance>
 </instances>
@@
 <junction x="111.76" y="71.12"/>
 </segment>
+<segment>
+<pinref part="C32" gate="G$1" pin="2"/>
+<pinref part="VSS53" gate="G$1" pin="VSS"/>
+<junction x="223.52" y="114.3"/>
+</segment>
 </net>
 <net name="SDI1" class="0">
@@
 <junction x="193.04" y="121.92"/>
 <junction x="193.04" y="116.84"/>
+<pinref part="C32" gate="G$1" pin="1"/>
+<wire x1="210.82" y1="121.92" x2="223.52" y2="121.92" width="0.1524" layer="91"/>
+<junction x="223.52" y="121.92"/>
 </segment>
 <segment>
@@
 <label x="114.3" y="86.36" size="1.778" layer="95"/>
 </segment>
+<segment>
+<wire x1="154.94" y1="58.42" x2="154.94" y2="66.04" width="0.1524" layer="91"/>
+<pinref part="R15" gate="G$1" pin="1"/>
+<junction x="154.94" y="66.04"/>
+<junction x="154.94" y="58.42"/>
+<label x="154.94" y="63.5" size="1.778" layer="95"/>
+</segment>
 </net>
 <net name="MA+" class="0">
@@
 <junction x="119.38" y="83.82"/>
 </segment>
+<segment>
+<wire x1="165.1" y1="58.42" x2="165.1" y2="66.04" width="0.1524" layer="91"/>
+<pinref part="R15" gate="G$1" pin="2"/>
+<junction x="165.1" y="58.42"/>
+<junction x="165.1" y="66.04"/>
+<label x="165.1" y="63.5" size="1.778" layer="95"/>
+</segment>
 </net>
 <net name="MO-" class="0">
@@
 <label x="114.3" y="81.28" size="1.778" layer="95"/>
 </segment>
+<segment>
+<wire x1="170.18" y1="58.42" x2="170.18" y2="66.04" width="0.1524" layer="91"/>
+<pinref part="R16" gate="G$1" pin="1"/>
+<junction x="170.18" y="66.04"/>
+<junction x="170.18" y="58.42"/>
+<label x="170.18" y="63.5" size="1.778" layer="95"/>
+</segment>
 </net>
 <net name="MO+" class="0">
@@
 <label x="114.3" y="78.74" size="1.778" layer="95"/>
 </segment>
+<segment>
+<wire x1="180.34" y1="58.42" x2="180.34" y2="66.04" width="0.1524" layer="91"/>
+<pinref part="R16" gate="G$1" pin="2"/>
+<junction x="180.34" y="58.42"/>
+<junction x="180.34" y="66.04"/>
+<label x="180.34" y="63.5" size="1.778" layer="95"/>
+</segment>
 </net>
 <net name="SL-" class="0">
@@
 <label x="114.3" y="91.44" size="1.778" layer="95"/>
 </segment>
+<segment>
+<wire x1="139.7" y1="66.04" x2="139.7" y2="58.42" width="0.1524" layer="91"/>
+<pinref part="R14" gate="G$1" pin="1"/>
+<junction x="139.7" y="58.42"/>
+<junction x="139.7" y="66.04"/>
+<label x="139.7" y="63.5" size="1.778" layer="95"/>
+</segment>
 </net>
 <net name="SL+" class="0">
@@
 <label x="114.3" y="88.9" size="1.778" layer="95"/>
 </segment>
+<segment>
+<wire x1="149.86" y1="66.04" x2="149.86" y2="58.42" width="0.1524" layer="91"/>
+<pinref part="R14" gate="G$1" pin="2"/>
+<junction x="149.86" y="66.04"/>
+<junction x="149.86" y="58.42"/>
+<label x="149.86" y="63.5" size="1.778" layer="95"/>
+</segment>
 </net>
 <net name="N$19" class="0">
@@
 <label x="121.92" y="76.2" size="1.778" layer="95"/>
 </segment>
+<segment>
+<wire x1="121.92" y1="66.04" x2="121.92" y2="58.42" width="0.1524" layer="91"/>
+<pinref part="R17" gate="G$1" pin="1"/>
+<junction x="121.92" y="58.42"/>
+<junction x="121.92" y="66.04"/>
+<label x="114.3" y="68.58" size="1.778" layer="95"/>
+</segment>
 </net>
 <net name="RS422_I+" class="0">
@@
 <label x="121.92" y="73.66" size="1.778" layer="95"/>
 </segment>
-</net>
+<segment>
+<wire x1="132.08" y1="66.04" x2="132.08" y2="58.42" width="0.1524" layer="91"/>
+<pinref part="R17" gate="G$1" pin="2"/>
+<junction x="132.08" y="58.42"/>
+<junction x="132.08" y="66.04"/>
+<label x="127" y="68.58" size="1.778" layer="95"/>
+</segment>
+</net>

Commit message: up
Parts:
- added D1: 5.6V, diode:DIODE-SMB
Connections:
- net VIN: now also D1.C
- net VSS: now also D1.A
Changed lines of the file:
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@@
 <layer number="97" name="Info" color="7" fill="1" visible="yes" active="yes"/>
 <layer number="98" name="Guide" color="6" fill="1" visible="yes" active="yes"/>
+<layer number="99" name="SpiceOrder" color="5" fill="1" visible="yes" active="yes"/>
 </layers>
 <schematic xreflabel="%F%N/%S.%C%R" xrefpart="/%S.%C%R">
@@
 </class>
 <class number="1" name="current" width="0.2032" drill="0">
+</class>
+<class number="2" name="high_current" width="0.3048" drill="0">
 </class>
 </classes>
@@
 <part name="C32" library="rcl" library_urn="urn:adsk.eagle:library:334" deviceset="C-US" device="C0805" package3d_urn="urn:adsk.eagle:package:23617/2" value="10uf"/>
 <part name="VSS53" library="supply1" library_urn="urn:adsk.eagle:library:371" deviceset="VSS" device=""/>
+<part name="D1" library="diode" library_urn="urn:adsk.eagle:library:210" deviceset="DIODE-" device="SMB" package3d_urn="urn:adsk.eagle:package:43404/2" value="5.6V"/>
+<part name="VSS54" library="supply1" library_urn="urn:adsk.eagle:library:371" deviceset="VSS" device=""/>
 </parts>
 <sheets>
@@
 <instance part="VSS53" gate="G$1" x="223.52" y="111.76" smashed="yes">
 <attribute name="VALUE" x="220.98" y="111.76" size="1.778" layer="96" rot="R180"/>
+</instance>
+<instance part="D1" gate="G$1" x="104.14" y="-78.74" smashed="yes" rot="R180">
+<attribute name="NAME" x="101.6" y="-79.2226" size="1.778" layer="95" rot="R180"/>
+<attribute name="VALUE" x="101.6" y="-76.4286" size="1.778" layer="96" rot="R180"/>
+</instance>
+<instance part="VSS54" gate="G$1" x="106.68" y="-81.28" smashed="yes">
+<attribute name="VALUE" x="104.14" y="-81.28" size="1.778" layer="96" rot="R180"/>
 </instance>
 </instances>
@@
 <junction x="223.52" y="114.3"/>
 </segment>
+<segment>
+<pinref part="D1" gate="G$1" pin="A"/>
+<pinref part="VSS54" gate="G$1" pin="VSS"/>
+<junction x="106.68" y="-78.74"/>
+</segment>
 </net>
 <net name="SDI1" class="0">
@@
 <label x="114.3" y="93.98" size="1.778" layer="95"/>
 </segment>
+<segment>
+<wire x1="101.6" y1="-78.74" x2="96.52" y2="-78.74" width="0.1524" layer="91"/>
+<pinref part="D1" gate="G$1" pin="C"/>
+<junction x="101.6" y="-78.74"/>
+<junction x="96.52" y="-78.74"/>
+<label x="96.52" y="-76.2" size="1.778" layer="95"/>
+</segment>
 </net>
 <net name="PGD" class="0">
@@
 </segment>
 </net>
-<net name="VIN_PWR" class="1">
+<net name="VIN_PWR" class="2">
 <segment>
 <pinref part="VIN_5+" gate="-2" pin="S"/>

Commit message: up
Parts:
- added C33, C34: 0.1uf, rcl:C-USC0603
Connections:
- net SW1: now also C33.1
- net SW2: now also C34.1
- net VSS: now also C33.2, C34.2
Changed lines of the file:
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@@
 <part name="D1" library="diode" library_urn="urn:adsk.eagle:library:210" deviceset="DIODE-" device="SMB" package3d_urn="urn:adsk.eagle:package:43404/2" value="5.6V"/>
 <part name="VSS54" library="supply1" library_urn="urn:adsk.eagle:library:371" deviceset="VSS" device=""/>
+<part name="C33" library="rcl" library_urn="urn:adsk.eagle:library:334" deviceset="C-US" device="C0603" package3d_urn="urn:adsk.eagle:package:23616/2" value="0.1uf"/>
+<part name="C34" library="rcl" library_urn="urn:adsk.eagle:library:334" deviceset="C-US" device="C0603" package3d_urn="urn:adsk.eagle:package:23616/2" value="0.1uf"/>
+<part name="VSS55" library="supply1" library_urn="urn:adsk.eagle:library:371" deviceset="VSS" device=""/>
+<part name="VSS56" library="supply1" library_urn="urn:adsk.eagle:library:371" deviceset="VSS" device=""/>
 </parts>
 <sheets>
@@
 <instance part="VSS54" gate="G$1" x="106.68" y="-81.28" smashed="yes">
 <attribute name="VALUE" x="104.14" y="-81.28" size="1.778" layer="96" rot="R180"/>
+</instance>
+<instance part="C33" gate="G$1" x="363.22" y="35.56" smashed="yes" rot="MR0">
+<attribute name="NAME" x="362.204" y="36.195" size="1.778" layer="95" rot="MR0"/>
+<attribute name="VALUE" x="362.204" y="31.369" size="1.778" layer="96" rot="MR0"/>
+</instance>
+<instance part="C34" gate="G$1" x="363.22" y="20.32" smashed="yes" rot="MR0">
+<attribute name="NAME" x="362.204" y="20.955" size="1.778" layer="95" rot="MR0"/>
+<attribute name="VALUE" x="362.204" y="16.129" size="1.778" layer="96" rot="MR0"/>
+</instance>
+<instance part="VSS55" gate="G$1" x="363.22" y="27.94" smashed="yes">
+<attribute name="VALUE" x="365.76" y="25.4" size="1.778" layer="96" rot="R180"/>
+</instance>
+<instance part="VSS56" gate="G$1" x="363.22" y="12.7" smashed="yes">
+<attribute name="VALUE" x="365.76" y="10.16" size="1.778" layer="96" rot="R180"/>
 </instance>
 </instances>
@@
 <junction x="106.68" y="-78.74"/>
 </segment>
+<segment>
+<pinref part="C33" gate="G$1" pin="2"/>
+<pinref part="VSS55" gate="G$1" pin="VSS"/>
+<junction x="363.22" y="30.48"/>
+</segment>
+<segment>
+<pinref part="C34" gate="G$1" pin="2"/>
+<pinref part="VSS56" gate="G$1" pin="VSS"/>
+<junction x="363.22" y="15.24"/>
+</segment>
 </net>
 <net name="SDI1" class="0">
@@
 <junction x="363.22" y="38.1"/>
 <label x="365.76" y="38.1" size="1.778" layer="95"/>
+<pinref part="C33" gate="G$1" pin="1"/>
 </segment>
 <segment>
@@
 <junction x="363.22" y="22.86"/>
 <label x="365.76" y="22.86" size="1.778" layer="95"/>
-</segment>
-<segment>
+<pinref part="C34" gate="G$1" pin="1"/>
+</segment>
+<segment>

Commit message: up
Parts:
- R1: value 100 ohm -> 56 ohm
- R11: value 50 ohm -> 120 ohm
- R3, R4, R5, R6: value 1K ohm -> 2.2K ohm
Changed lines of the file:
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@@
 <part name="VDD4" library="supply1" library_urn="urn:adsk.eagle:library:371" deviceset="VDD" device=""/>
 <part name="VSS10" library="supply1" library_urn="urn:adsk.eagle:library:371" deviceset="VSS" device=""/>
-<part name="R1" library="rcl" library_urn="urn:adsk.eagle:library:334" deviceset="R-US_" device="R0805" package3d_urn="urn:adsk.eagle:package:23553/2" value="100 ohm"/>
+<part name="R1" library="rcl" library_urn="urn:adsk.eagle:library:334" deviceset="R-US_" device="R0805" package3d_urn="urn:adsk.eagle:package:23553/2" value="56 ohm"/>
 <part name="R2" library="rcl" library_urn="urn:adsk.eagle:library:334" deviceset="R-US_" device="R0805" package3d_urn="urn:adsk.eagle:package:23553/2" value="10K ohm"/>
 <part name="C16" library="rcl" library_urn="urn:adsk.eagle:library:334" deviceset="C-US" device="C0603" package3d_urn="urn:adsk.eagle:package:23616/2" value="1000pf"/>
@@
 <part name="VDD9" library="supply1" library_urn="urn:adsk.eagle:library:371" deviceset="VDD" device=""/>
 <part name="ICSP" library="pinhead" library_urn="urn:adsk.eagle:library:325" deviceset="PINHD-1X6" device="/90" package3d_urn="urn:adsk.eagle:package:22475/2" value="ICSP"/>
-<part name="R3" library="rcl" library_urn="urn:adsk.eagle:library:334" deviceset="R-US_" device="R0805" package3d_urn="urn:adsk.eagle:package:23553/2" value="1K ohm"/>
+<part name="R3" library="rcl" library_urn="urn:adsk.eagle:library:334" deviceset="R-US_" device="R0805" package3d_urn="urn:adsk.eagle:package:23553/2" value="2.2K ohm"/>
 <part name="VDD10" library="supply1" library_urn="urn:adsk.eagle:library:371" deviceset="VDD" device=""/>
 <part name="POWER" library="led" library_urn="urn:adsk.eagle:library:259" deviceset="LED" device="CHIP-LED0603" package3d_urn="urn:adsk.eagle:package:15819/3" value="POWER"/>
@@
 <part name="VSS18" library="supply1" library_urn="urn:adsk.eagle:library:371" deviceset="VSS" device=""/>
 <part name="VSS19" library="supply1" library_urn="urn:adsk.eagle:library:371" deviceset="VSS" device=""/>
-<part name="R4" library="rcl" library_urn="urn:adsk.eagle:library:334" deviceset="R-US_" device="R0805" package3d_urn="urn:adsk.eagle:package:23553/2" value="1K ohm"/>
-<part name="R5" library="rcl" library_urn="urn:adsk.eagle:library:334" deviceset="R-US_" device="R0805" package3d_urn="urn:adsk.eagle:package:23553/2" value="1K ohm"/>
-<part name="R6" library="rcl" library_urn="urn:adsk.eagle:library:334" deviceset="R-US_" device="R0805" package3d_urn="urn:adsk.eagle:package:23553/2" value="1K ohm"/>
+<part name="R4" library="rcl" library_urn="urn:adsk.eagle:library:334" deviceset="R-US_" device="R0805" package3d_urn="urn:adsk.eagle:package:23553/2" value="2.2K ohm"/>
+<part name="R5" library="rcl" library_urn="urn:adsk.eagle:library:334" deviceset="R-US_" device="R0805" package3d_urn="urn:adsk.eagle:package:23553/2" value="2.2K ohm"/>
+<part name="R6" library="rcl" library_urn="urn:adsk.eagle:library:334" deviceset="R-US_" device="R0805" package3d_urn="urn:adsk.eagle:package:23553/2" value="2.2K ohm"/>
 <part name="MISC_ANA" library="pinhead" library_urn="urn:adsk.eagle:library:325" deviceset="PINHD-1X6" device="/90" package3d_urn="urn:adsk.eagle:package:22475/2" value="MISC_ANA"/>
 <part name="VIN_5+" library="con-molex" library_urn="urn:adsk.eagle:library:165" deviceset="22-23-2021" device="" package3d_urn="urn:adsk.eagle:package:8078633/1"/>
@@
 <part name="USBC-PWR" library="con-lstb" library_urn="urn:adsk.eagle:library:162" deviceset="MA04-1" device="" package3d_urn="urn:adsk.eagle:package:8337/1" value="USBC-PWR"/>
 <part name="VSS43" library="supply1" library_urn="urn:adsk.eagle:library:371" deviceset="VSS" device=""/>
-<part name="R11" library="rcl" library_urn="urn:adsk.eagle:library:334" deviceset="R-US_" device="R0603" package3d_urn="urn:adsk.eagle:package:23555/3" value="50 ohm"/>
+<part name="R11" library="rcl" library_urn="urn:adsk.eagle:library:334" deviceset="R-US_" device="R0603" package3d_urn="urn:adsk.eagle:package:23555/3" value="120 ohm"/>
 <part name="R12" library="rcl" library_urn="urn:adsk.eagle:library:334" deviceset="R-US_" device="R0603" package3d_urn="urn:adsk.eagle:package:23555/3" value="50 ohm"/>
 <part name="R13" library="rcl" library_urn="urn:adsk.eagle:library:334" deviceset="R-US_" device="R0603" package3d_urn="urn:adsk.eagle:package:23555/3" value="50 ohm"/>
